Commit message: Added the logic needed to read/write to a mounted robotiq gripper

File: link6_description/urdf/kortex3.ros2control.xacro (robot description, xacro)
@@ -44,4 +44,9 @@
         <state_interface name="effort"/>
     </joint>
+    <joint name="robotiq_85_left_knuckle_joint">
+        <command_interface name="position" />
+        <state_interface name="position"/>
+        <state_interface name="velocity"/>
+    </joint>
 </ros2_control>
 </robot>
