Commit message: Added the gripper to robot's description (can be visualized in rviz now)

File: link6_description/urdf/link6_calibrated.xacro (robot description, xacro)
@@ -380,3 +380,41 @@
         <limit lower="0" upper="0" effort="0" velocity="0"/>
     </joint>
+    <!-- Include and load the gripper if defined -->
+    <!--
+    <xacro:unless value="${not gripper}">
+    <xacro:include filename="$(find kortex_description)/grippers/${gripper}/urdf/${gripper}_macro.xacro" />
+    -->
+      <xacro:include filename="$(find robotiq_description)/urdf/robotiq_2f_85_macro.urdf.xacro" />
+      <!-- last_arm_link is defined in "$(find kortex_description)/arms/${arm}/urdf/${arm}_macro.xacro" -->
+      <!--
+    <xacro:robotiq_gripper
+        name="${prefix}RobotiqGripperHardwareInterface"
+        prefix="${prefix}"
+        parent="${parent}"
+        include_ros2_control="${include_ros2_control}"
+        com_port="${com_port}"
+        use_fake_hardware="${use_fake_hardware}"
+        fake_sensor_commands="${fake_sensor_commands}"
+        sim_ignition="${sim_ignition}"
+        sim_isaac="${sim_isaac}"
+        isaac_joint_commands="${isaac_joint_commands}"
+        isaac_joint_states="${isaac_joint_states}">
+        <origin xyz="0 0 0" rpy="0 0 0" />
+    </xacro:robotiq_gripper>
+    </xacro:unless>
+    -->
+    <xacro:robotiq_gripper
+        name="RobotiqGripperHardwareInterface"
+        prefix=""
+        parent="end_effector_link"
+        include_ros2_control="false"
+        com_port="/dev/ttyUSB0"
+        use_fake_hardware="false"
+        fake_sensor_commands="false"
+        sim_ignition="false"
+        sim_isaac="false"
+        isaac_joint_commands="/isaac_joint_commands"
+        isaac_joint_states="/isaac_joint_states">
+        <origin xyz="0 0 0" rpy="0 0 0" />
+    </xacro:robotiq_gripper>
 </robot>
