Commit message: Added the option to mounted/unmount the gripper

File: link6_description/urdf/link6.xacro (robot description, xacro)
@@ -1,5 +1,8 @@
 <?xml version="1.0" encoding="UTF-8" ?>
 <robot name="link6" xmlns:xacro="http://ros.org/wiki/xacro">
+    <!-- Arguments -->
+    <xacro:arg name="gripper" default="" />
     <xacro:include filename="$(find link6_description)/urdf/link6_calibrated.xacro" />
     <xacro:include filename="$(find link6_description)/urdf/kortex3.ros2control.xacro" />
+    <xacro:load_robot gripper="$(arg gripper)"/>
 </robot>

File: link6_description/urdf/link6_calibrated.xacro (robot description, xacro)
@@ -1,4 +1,5 @@
 <?xml version="1.0" encoding="utf-8"?>
 <robot name="link6_calibrated_old" xmlns:xacro="http://ros.org/wiki/xacro">
+<xacro:macro name="load_robot" params="gripper">
     <material name="lightgray">
         <color rgba="0.5294117647058824 0.5294117647058824 0.5294117647058824 1"/>
@@ -380,41 +381,32 @@
         <limit lower="0" upper="0" effort="0" velocity="0"/>
     </joint>
+    <!-- If no gripper, define tool frame here -->
+    <xacro:if value="${not gripper}">
+      <link name="tool_frame"/>
+      <joint name="tool_frame_joint" type="fixed">
+        <origin xyz="0 0 0" rpy="0 0 0" />
+        <parent link="end_effector_link" />
+        <child link="tool_frame" />
+        <axis xyz="0 0 0" />
+      </joint>
+    </xacro:if>
     <!-- Include and load the gripper if defined -->
-    <!--
     <xacro:unless value="${not gripper}">
-    <xacro:include filename="$(find kortex_description)/grippers/${gripper}/urdf/${gripper}_macro.xacro" />
-    -->
-      <xacro:include filename="$(find robotiq_description)/urdf/robotiq_2f_85_macro.urdf.xacro" />
-      <!-- last_arm_link is defined in "$(find kortex_description)/arms/${arm}/urdf/${arm}_macro.xacro" -->
-      <!--
-    <xacro:robotiq_gripper
-        name="${prefix}RobotiqGripperHardwareInterface"
-        prefix="${prefix}"
-        parent="${parent}"
-        include_ros2_control="${include_ros2_control}"
-        com_port="${com_port}"
-        use_fake_hardware="${use_fake_hardware}"
-        fake_sensor_commands="${fake_sensor_commands}"
-        sim_ignition="${sim_ignition}"
-        sim_isaac="${sim_isaac}"
-        isaac_joint_commands="${isaac_joint_commands}"
-        isaac_joint_states="${isaac_joint_states}">
-        <origin xyz="0 0 0" rpy="0 0 0" />
-    </xacro:robotiq_gripper>
+        <xacro:include filename="$(find robotiq_description)/urdf/robotiq_2f_85_macro.urdf.xacro" />
+        <xacro:robotiq_gripper
+            name="RobotiqGripperHardwareInterface"
+            prefix=""
+            parent="end_effector_link"
+            include_ros2_control="false"
+            com_port="/dev/ttyUSB0"
+            use_fake_hardware="false"
+            fake_sensor_commands="false"
+            sim_ignition="false"
+            sim_isaac="false"
+            isaac_joint_commands="/isaac_joint_commands"
+            isaac_joint_states="/isaac_joint_states">
+            <origin xyz="0 0 0" rpy="0 0 0" />
+        </xacro:robotiq_gripper>
     </xacro:unless>
-    -->
-    <xacro:robotiq_gripper
-        name="RobotiqGripperHardwareInterface"
-        prefix=""
-        parent="end_effector_link"
-        include_ros2_control="false"
-        com_port="/dev/ttyUSB0"
-        use_fake_hardware="false"
-        fake_sensor_commands="false"
-        sim_ignition="false"
-        sim_isaac="false"
-        isaac_joint_commands="/isaac_joint_commands"
-        isaac_joint_states="/isaac_joint_states">
-        <origin xyz="0 0 0" rpy="0 0 0" />
-    </xacro:robotiq_gripper>
+    </xacro:macro>
 </robot>
