Commit message: Integrated the robotiq_2f_85 gripper in Gazebo simulation

File: link6_description/urdf/link6_gz.urdf.xacro (robot description, xacro)
@@ -1,4 +1,7 @@
 <?xml version="1.0" encoding="utf-8"?>
-<robot name="link6" version="1.0">
+<robot name="link6" version="1.0" xmlns:xacro="http://www.ros.org/wiki/xacro">
+  <!-- Arguments -->
+  <xacro:arg name="gripper" default="" />
+  <!--<xacro:property name="gripper_prop" value="$(arg gripper)"/>-->
   <material name="lightgray">
     <color rgba="0.5294117647058824 0.5294117647058824 0.5294117647058824 1"/>
@@ -224,4 +227,32 @@
     <limit lower="0" upper="0" effort="0" velocity="0"/>
   </joint>
+    <!-- If no gripper, define tool frame here -->
+    <xacro:unless value="${'$(arg gripper)' != ''}">
+      <link name="tool_frame"/>
+      <joint name="tool_frame_joint" type="fixed">
+        <origin xyz="0 0 0" rpy="0 0 0" />
+        <parent link="end_effector_link" />
+        <child link="tool_frame" />
+        <axis xyz="0 0 0" />
+      </joint>
+    </xacro:unless>
+    <!-- Include and load the gripper if defined -->
+    <xacro:if value="${'$(arg gripper)' != ''}">
+        <xacro:include filename="$(find robotiq_description)/urdf/robotiq_2f_85_macro.urdf.xacro" />
+        <xacro:robotiq_gripper
+            name="RobotiqGripperHardwareInterface"
+            prefix=""
+            parent="end_effector_link"
+            include_ros2_control="true"
+            com_port="/dev/ttyUSB0"
+            use_fake_hardware="false"
+            fake_sensor_commands="false"
+            sim_ignition="true"
+            sim_isaac="false"
+            isaac_joint_commands="/isaac_joint_commands"
+            isaac_joint_states="/isaac_joint_states">
+            <origin xyz="0 0 0" rpy="0 0 0" />
+        </xacro:robotiq_gripper>
+    </xacro:if>
   <ros2_control name="Link6GzSim" type="system">
     <hardware>
