Commit message: fixed macros so that left is true left and right is true right gripper

File: link6_description/urdf/double_robotiq_90_macro.urdf.xacro (robot description, xacro)
@@ -32,10 +32,10 @@
         </joint>
         <joint name="${prefix}left_gripper_joint" type="fixed">
-            <origin xyz="0.025 0.025 0.075" rpy="${PI/2} 0.0 ${PI/4}"/>
+            <origin xyz="-0.025 0.025 0.075" rpy="${PI/2} 0.0 ${-PI/4}"/>
             <parent link="${prefix}double_gripper_base_link"/>
             <child link="${prefix}left_gripper_link"/>
         </joint>
         <joint name="${prefix}right_gripper_joint" type="fixed">
-            <origin xyz="-0.025 0.025 0.075" rpy="${PI/2} 0.0 ${-PI/4}"/>
+            <origin xyz="0.025 0.025 0.075" rpy="${PI/2} 0.0 ${PI/4}"/>
             <parent link="${prefix}double_gripper_base_link"/>
             <child link="${prefix}right_gripper_link"/>

File: link6_description/urdf/double_robotiq_macro.urdf.xacro (robot description, xacro)
@@ -32,10 +32,10 @@
         </joint>
         <joint name="${prefix}left_gripper_joint" type="fixed">
-            <origin xyz="0.0 0.0 0.0" rpy="0.0 ${PI/4} 0.0"/>
+            <origin xyz="0.0 0.0 0.0" rpy="0.0 ${-PI/4} 0.0"/>
             <parent link="${prefix}double_gripper_base_link"/>
             <child link="${prefix}left_gripper_link"/>
         </joint>
         <joint name="${prefix}right_gripper_joint" type="fixed">
-            <origin xyz="0.0 0.0 0.0" rpy="0.0 ${-PI/4} 0.0"/>
+            <origin xyz="0.0 0.0 0.0" rpy="0.0 ${PI/4} 0.0"/>
             <parent link="${prefix}double_gripper_base_link"/>
             <child link="${prefix}right_gripper_link"/>
@@ -51,5 +51,5 @@
             sim_ignition="${use_sim}"
             com_port="${gripper_com_port_left}">
-            <origin xyz="0 0 0.5" rpy="0 0 0"/>
+            <origin xyz="0 0 0.1" rpy="0 0 0"/>
         </xacro:robotiq_gripper>
         <!-- Include right gripper -->
@@ -63,5 +63,5 @@
             sim_ignition="${use_sim}"
             com_port="${gripper_com_port_right}">
-            <origin xyz="0 0 0.5" rpy="0 0 0"/>
+            <origin xyz="0 0 0.1" rpy="0 0 0"/>
         </xacro:robotiq_gripper>
     </xacro:macro>

Commit message: Added tool frames for both grippers

File: link6_description/urdf/double_robotiq_90_macro.urdf.xacro (robot description, xacro)
@@ -12,31 +12,26 @@
         <xacro:property name="PI" value="3.14159"/>
         <xacro:include filename="$(find robotiq_description)/urdf/robotiq_2f_85_macro.urdf.xacro"/>
-        <link name="${prefix}double_gripper_base_link">
-            <visual>
-                <geometry>
-                    <box size="0.01 0.01 0.01"/>
-                </geometry>
-            </visual>
-            <collision>
-                <geometry>
-                    <sphere radius="0.02"/>
-                </geometry>
-            </collision>
-        </link>
+        <link name="${prefix}double_gripper_90_degrees_angle_bracket"></link>
+        <joint name="${prefix}double_gripper_90_degrees_angle_bracket_joint" type="fixed">
+            <parent link="${parent}"/>
+            <child link="${prefix}double_gripper_90_degrees_angle_bracket"/>
+            <xacro:insert_block name="origin" />
+        </joint>
+        <link name="${prefix}double_gripper_mount_link"></link>
+        <joint name="${prefix}double_gripper_mount_joint" type="fixed">
+            <origin xyz="0 0.0255 0.063" rpy="${PI/2} 0 0"/>
+            <parent link="${prefix}double_gripper_90_degrees_angle_bracket"/>
+            <child link="${prefix}double_gripper_mount_link"/>
+        </joint>
         <link name="${prefix}left_gripper_link"/>
         <link name="${prefix}right_gripper_link"/>
-        <joint name="${prefix}double_gripper_base_joint" type="fixed">
-            <parent link="${parent}"/>
-            <child link="${prefix}double_gripper_base_link"/>
-            <xacro:insert_block name="origin" />
-        </joint>
         <joint name="${prefix}left_gripper_joint" type="fixed">
-            <origin xyz="0.025 0.025 0.075" rpy="${PI/2} 0.0 ${PI/4}"/>
-            <parent link="${prefix}double_gripper_base_link"/>
+            <origin xyz="-0.042 0 0.036" rpy="0 -${PI/6} 0"/>
+            <parent link="${prefix}double_gripper_mount_link"/>
             <child link="${prefix}left_gripper_link"/>
         </joint>
         <joint name="${prefix}right_gripper_joint" type="fixed">
-            <origin xyz="-0.025 0.025 0.075" rpy="${PI/2} 0.0 ${-PI/4}"/>
-            <parent link="${prefix}double_gripper_base_link"/>
+            <origin xyz="0.042 0 0.036" rpy="0 ${PI/6} 0"/>
+            <parent link="${prefix}double_gripper_mount_link"/>
             <child link="${prefix}right_gripper_link"/>
         </joint>
@@ -51,6 +46,12 @@
             sim_ignition="${use_sim}"
             com_port="${gripper_com_port_left}">
-            <origin xyz="0 0 0" rpy="0 0 0"/>
+            <origin xyz="0 0 0" rpy="0 0 ${PI}"/>
         </xacro:robotiq_gripper>
+        <link name="${prefix}left_tool_frame"></link>
+        <joint name="${prefix}left_tool_frame_joint" type="fixed">
+            <origin xyz="0 0 0.12" rpy="0 0 0"/>
+            <parent link="${prefix}left_robotiq_85_base_link"/>
+            <child link="${prefix}left_tool_frame"/>
+        </joint>
         <!-- Include right gripper -->
         <xacro:robotiq_gripper
@@ -63,6 +64,12 @@
             sim_ignition="${use_sim}"
             com_port="${gripper_com_port_right}">
-            <origin xyz="0 0 0" rpy="0 0 0"/>
+            <origin xyz="0 0 0" rpy="0 0 ${PI}"/>
         </xacro:robotiq_gripper>
+        <link name="${prefix}right_tool_frame"></link>
+        <joint name="${prefix}right_tool_frame_joint" type="fixed">
+            <origin xyz="0 0 0.12" rpy="0 0 0"/>
+            <parent link="${prefix}right_robotiq_85_base_link"/>
+            <child link="${prefix}right_tool_frame"/>
+        </joint>
     </xacro:macro>
 </robot>

Commit message: Started separating the gripper from the link6_macro

File: link6_description/urdf/double_robotiq_90_macro.urdf.xacro (robot description, xacro)
@@ -11,5 +11,12 @@
         com_port_right:=/dev/ttyUSB1">
         <xacro:property name="PI" value="3.14159"/>
-        <xacro:include filename="$(find robotiq_description)/urdf/robotiq_2f_85_macro.urdf.xacro"/>
+        <xacro:arg name="grip_pos_min" default="0"/>
+        <xacro:arg name="grip_pos_max" default="0.025"/>
+        <xacro:arg name="baudrate" default="115200"/>
+        <xacro:arg name="parity" default="N"/>
+        <xacro:arg name="data_bits" default="8"/>
+        <xacro:arg name="stop_bit" default="1"/>
+        <xacro:arg name="slave_id" default="9"/>
+        <xacro:include filename="$(find link6_description)/urdf/robotiq_hande_cutter.xacro"/>
         <link name="${prefix}double_gripper_90_degrees_angle_bracket"></link>
         <joint name="${prefix}double_gripper_90_degrees_angle_bracket_joint" type="fixed">
@@ -37,39 +44,41 @@
         </joint>
         <!-- Include left gripper -->
-        <xacro:robotiq_gripper
+        <xacro:robotiq_hande_gripper
             name="LeftRobotiqGripperHardwareInterface"
             prefix="${prefix}left_"
             parent="${prefix}left_gripper_link"
+            grip_pos_min="$(arg grip_pos_min)"
+            grip_pos_max="$(arg grip_pos_max)"
+            tty_port="${gripper_com_port_left}"
+            baudrate="$(arg baudrate)"
+            parity="$(arg parity)"
+            data_bits="$(arg data_bits)"
+            stop_bit="$(arg stop_bit)"
+            slave_id="$(arg slave_id)"
             use_fake_hardware="${use_fake_hardware}"
-            fake_sensor_commands="${fake_sensor_commands}"
             include_ros2_control="${sim_gazebo}"
-            sim_ignition="${use_sim}"
-            com_port="${gripper_com_port_left}">
-            <origin xyz="0 0 0" rpy="0 0 ${PI}"/>
-        </xacro:robotiq_gripper>
-        <link name="${prefix}left_tool_frame"></link>
-        <joint name="${prefix}left_tool_frame_joint" type="fixed">
-            <origin xyz="0 0 0.12" rpy="0 0 0"/>
-            <parent link="${prefix}left_robotiq_85_base_link"/>
-            <child link="${prefix}left_tool_frame"/>
-        </joint>
+            sim_gazebo="${sim_gazebo}"
+            xyz="0 0 0"
+            rpy="0 0 ${PI}"
+        />
         <!-- Include right gripper -->
-        <xacro:robotiq_gripper
+        <xacro:robotiq_hande_gripper
             name="RightRobotiqGripperHardwareInterface"
             prefix="${prefix}right_"
             parent="${prefix}right_gripper_link"
+            grip_pos_min="$(arg grip_pos_min)"
+            grip_pos_max="$(arg grip_pos_max)"
+            tty_port="${gripper_com_port_right}"
+            baudrate="$(arg baudrate)"
+            parity="$(arg parity)"
+            data_bits="$(arg data_bits)"
+            stop_bit="$(arg stop_bit)"
+            slave_id="$(arg slave_id)"
             use_fake_hardware="${use_fake_hardware}"
-            fake_sensor_commands="${fake_sensor_commands}"
             include_ros2_control="${sim_gazebo}"
-            sim_ignition="${use_sim}"
-            com_port="${gripper_com_port_right}">
-            <origin xyz="0 0 0" rpy="0 0 ${PI}"/>
-        </xacro:robotiq_gripper>
-        <link name="${prefix}right_tool_frame"></link>
-        <joint name="${prefix}right_tool_frame_joint" type="fixed">
-            <origin xyz="0 0 0.12" rpy="0 0 0"/>
-            <parent link="${prefix}right_robotiq_85_base_link"/>
-            <child link="${prefix}right_tool_frame"/>
-        </joint>
+            sim_gazebo="${sim_gazebo}"
+            xyz="0 0 0"
+            rpy="0 0 ${PI}"
+        />
     </xacro:macro>
 </robot>

File: link6_description/urdf/link6.ros2_control.xacro (robot description, xacro)
@@ -4,4 +4,5 @@
     params="
     prefix
+    gripper
     use_fake_hardware:=false
     fake_sensor_commands:=false
@@ -111,14 +112,30 @@
       </joint>
       <xacro:unless value="${sim_gazebo}">
-        <joint name="${prefix}right_robotiq_85_left_knuckle_joint">
-          <command_interface name="position" />
-          <state_interface name="position" />
-          <state_interface name="velocity" />
-        </joint>
-        <joint name="${prefix}left_robotiq_85_left_knuckle_joint">
-          <command_interface name="position" />
-          <state_interface name="position" />
-          <state_interface name="velocity" />
-        </joint>
+        <xacro:if value="${gripper == 'robotiq_2f_85'}">
+          <joint name="${prefix}robotiq_85_left_knuckle_joint">
+            <command_interface name="position" />
+            <state_interface name="position" />
+            <state_interface name="velocity" />
+          </joint>
+        </xacro:if>
+        <xacro:if value="${gripper == 'robotiq_hande'}">
+          <joint name="${prefix}robotiq_hande_left_finger_joint">
+            <command_interface name="position" />
+            <state_interface name="position" />
+            <state_interface name="velocity" />
+          </joint>
+        </xacro:if>
+        <xacro:if value="${gripper == 'double_robotiq_90'}">
+          <joint name="${prefix}right_robotiq_hande_left_finger_joint">
+            <command_interface name="position" />
+            <state_interface name="position" />
+            <state_interface name="velocity" />
+          </joint>
+          <joint name="${prefix}left_robotiq_hande_left_finger_joint">
+            <command_interface name="position" />
+            <state_interface name="position" />
+            <state_interface name="velocity" />
+          </joint>
+        </xacro:if>
       </xacro:unless>
     </ros2_control>

File: link6_description/urdf/link6_macro.xacro (robot description, xacro)
@@ -20,4 +20,5 @@
     <xacro:link6_ros2_control
       prefix="${prefix}"
+      gripper="${gripper}"
       use_fake_hardware="${use_fake_hardware}"
       fake_sensor_commands="${fake_sensor_commands}"
@@ -446,4 +447,25 @@
       </joint>
     </xacro:if>
+    <xacro:if value="${gripper == 'robotiq_hande'}">
+      <xacro:include filename="$(find link6_description)/urdf/robotiq_hande_cutter.xacro" />
+      <xacro:robotiq_hande_gripper
+          name="RobotiqGripperHardwareInterface"
+          prefix="${prefix}"
+          parent="${prefix}end_effector_link"
+          grip_pos_min="0"
+          grip_pos_max="0.025"
+          tty_port="${gripper_com_port_left}"
+          baudrate="115200"
+          parity="N"
+          data_bits="8"
+          stop_bit="1"
+          slave_id="9"
+          use_fake_hardware="${use_fake_hardware}"
+          include_ros2_control="${sim_gazebo}"
+          sim_gazebo="${sim_gazebo}"
+          xyz="0 0 0"
+          rpy="0 0 3.14159"
+      />
+    </xacro:if>
     <xacro:if value="${gripper == 'double_robotiq'}">
       <xacro:include filename="$(find link6_description)/urdf/double_robotiq_macro.urdf.xacro" />

File: link6_description/urdf/link6_robotiq_2f_85.urdf.xacro (robot description, xacro)
@@ -6,17 +6,9 @@
     <xacro:arg name="password" default="admin" />
     <xacro:arg name="port" default="10000" />
-    <xacro:arg name="port_realtime" default="10001" />
-    <xacro:arg name="session_inactivity_timeout_ms" default="60000" />
-    <xacro:arg name="connection_inactivity_timeout_ms" default="2000" />
-    <xacro:arg name="gripper" default="" />
-    <xacro:arg name="gripper_joint_name" default="finger_joint" />
-    <xacro:arg name="gripper_max_velocity" default="100.0" />
-    <xacro:arg name="gripper_max_force" default="100.0" />
     <xacro:arg name="sim_gazebo" default="false" />
     <xacro:arg name="prefix" default="" />
     <xacro:arg name="use_fake_hardware" default="false" />
     <xacro:arg name="fake_sensor_commands" default="false" />
-    <xacro:arg name="use_internal_bus_gripper_comm" default="false" />
-    <xacro:arg name="use_external_cable" default="false" />
+    <xacro:arg name="gripper_com_port" default="/dev/ttyUSB0" />
     <xacro:include filename="$(find link6_description)/urdf/link6_macro.xacro" />
     <!-- initial position for simulations (Mock Hardware, Gazebo) -->
@@ -39,15 +31,26 @@
         <origin xyz="0 0 0" rpy="0 0 0" />  <!-- position robot in the world -->
     </xacro:link6>
-    <link name="$(arg prefix)tool_frame" />
+    <!-- Include and load the gripper -->
+    <xacro:include filename="$(find robotiq_description)/urdf/robotiq_2f_85_macro.urdf.xacro" />
+    <xacro:robotiq_gripper
+        name="RobotiqGripperHardwareInterface"
+        parent="$(arg prefix)end_effector_link"
+        prefix="$(arg prefix)"
+        use_fake_hardware="$(arg use_fake_hardware)"
+        fake_sensor_commands="$(arg fake_sensor_commands)"
+        include_ros2_control="$(arg sim_gazebo)"
+        com_port="$(arg gripper_com_port)"
+        sim_ignition="$(arg sim_gazebo)">
+        <origin xyz="0 0 0" rpy="0 0 3.14159" />
+    </xacro:robotiq_gripper>
+    <link name="$(arg prefix)tool_frame"></link>
     <joint name="$(arg prefix)tool_frame_joint" type="fixed">
-        <origin xyz="0 0 0" rpy="0 0 0" />
-        <parent link="$(arg prefix)end_effector_link" />
-        <child link="$(arg prefix)tool_frame" />
-        <axis xyz="0 0 0" />
+        <origin xyz="0 0 0.12" rpy="0 0 0"/>
+        <parent link="$(arg prefix)robotiq_85_base_link"/>
+        <child link="$(arg prefix)tool_frame"/>
     </joint>
     <xacro:if value="$(arg sim_gazebo)">
         <gazebo>
-            <plugin filename="gz_ros2_control-system"
-                name="gz_ros2_control::GazeboSimROS2ControlPlugin">
+            <plugin filename="gz_ros2_control-system" name="gz_ros2_control::GazeboSimROS2ControlPlugin">
                 <parameters>$(find link6_control)/config/kortex3_controllers.yaml</parameters>
                 <controller_manager_node_name>controller_manager</controller_manager_node_name>
