Commit message: Added new calibration extraction procedure, which generates a parameter file instead of a full urdf

File: link6_description/urdf/link6.urdf.xacro (robot description, xacro)
@@ -19,10 +19,10 @@
     <xacro:arg name="use_internal_bus_gripper_comm" default="false" />
     <xacro:arg name="use_external_cable" default="false" />
+    <!-- Initial position for simulations (Mock Hardware, Gazebo) -->
+    <xacro:arg name="initial_positions_file" default="$(find link6_description)/config/initial_positions.yaml" />
+    <!-- Robot-specific calibration -->
+    <xacro:arg name="calibration_file" default="$(find link6_description)/config/default_calibration.yaml" />
+    <!-- Include Link6 macro -->
     <xacro:include filename="$(find link6_description)/urdf/link6_macro.xacro" />
-    <!-- initial position for simulations (Mock Hardware, Gazebo) -->
-    <xacro:arg name="initial_positions_file"
-        default="$(find link6_description)/config/initial_positions.yaml" />
-    <!-- convert to property to use substitution in function -->
-    <xacro:property name="initial_positions_file" default="$(arg initial_positions_file)" />
     <link name="world" />
     <xacro:link6
@@ -36,5 +36,6 @@
         fake_sensor_commands="$(arg fake_sensor_commands)"
         sim_gazebo="$(arg sim_gazebo)"
-        initial_positions="${xacro.load_yaml(initial_positions_file)}">
+        initial_positions_file="$(arg initial_positions_file)"
+        calibration_file="$(arg calibration_file)">
         <origin xyz="0 0 0" rpy="0 0 0" />  <!-- position robot in the world -->
     </xacro:link6>

File: link6_description/urdf/link6_macro.xacro (robot description, xacro)
@@ -13,8 +13,26 @@
     fake_sensor_commands:=false
     sim_gazebo:=false
-    initial_positions:=${dict(joint_1=0.0,joint_2=0.0,joint_3=0.0,joint_4=0.0,joint_5=0.0,joint_6=0.0)}
     gripper_com_port:=/dev/ttyUSB0
-    moveit_active:=false">
-    <!-- Properties -->
+    moveit_active:=false
+    initial_positions_file:='$(find link6_description)/config/initial_positions.yaml'
+    calibration_file:='$(find link6_description)/config/default_calibration.yaml'">
+    <!-- Load initial positions from yaml file -->
+    <xacro:property name="initial_positions" value="${xacro.load_yaml(initial_positions_file)}" />
+    <!-- Load calibration data from YAML file -->
+    <xacro:property name="calib" value="${xacro.load_yaml(calibration_file)}" />
+    <!-- Define joint origin properties from calibration data -->
+    <xacro:property name="joint_1_xyz" value="${calib['joint_1']['xyz']}" />
+    <xacro:property name="joint_1_rpy" value="${calib['joint_1']['rpy']}" />
+    <xacro:property name="joint_2_xyz" value="${calib['joint_2']['xyz']}" />
+    <xacro:property name="joint_2_rpy" value="${calib['joint_2']['rpy']}" />
+    <xacro:property name="joint_3_xyz" value="${calib['joint_3']['xyz']}" />
+    <xacro:property name="joint_3_rpy" value="${calib['joint_3']['rpy']}" />
+    <xacro:property name="joint_4_xyz" value="${calib['joint_4']['xyz']}" />
+    <xacro:property name="joint_4_rpy" value="${calib['joint_4']['rpy']}" />
+    <xacro:property name="joint_5_xyz" value="${calib['joint_5']['xyz']}" />
+    <xacro:property name="joint_5_rpy" value="${calib['joint_5']['rpy']}" />
+    <xacro:property name="joint_6_xyz" value="${calib['joint_6']['xyz']}" />
+    <xacro:property name="joint_6_rpy" value="${calib['joint_6']['rpy']}" />
+    <!-- Other properties -->
     <xacro:property name="base_collision_radius" value="0.08"/>
     <xacro:property name="shoulder_collision_radius" value="0.07"/>
@@ -119,5 +137,5 @@
     </link>
     <joint name="${prefix}joint_1" type="revolute">
-      <origin xyz="0 0 0.053" rpy="3.141592653589793 0 0" />
+      <origin xyz="${joint_1_xyz}" rpy="${joint_1_rpy}" />
       <parent link="${prefix}base_link" />
       <child link="${prefix}shoulder_link" />
@@ -208,5 +226,5 @@
     </link>
     <joint name="${prefix}joint_2" type="revolute">
-      <origin xyz="0.11024 -0.069257 -0.1375" rpy="-1.5707963267948966 0 0" />
+      <origin xyz="${joint_2_xyz}" rpy="${joint_2_rpy}" />
       <parent link="${prefix}shoulder_link" />
       <child link="${prefix}arm_link" />
@@ -261,5 +279,5 @@
     </link>
     <joint name="${prefix}joint_3" type="revolute">
-      <origin xyz="0 0.485 0" rpy="-3.141592653589793 0 0" />
+      <origin xyz="${joint_3_xyz}" rpy="${joint_3_rpy}" />
       <parent link="${prefix}arm_link" />
       <child link="${prefix}forearm_link" />
@@ -321,5 +339,5 @@
     </link>
     <joint name="${prefix}joint_4" type="revolute">
-      <origin xyz="0 -0.15216 -0.091704" rpy="-1.5707963267948966 0 0" />
+      <origin xyz="${joint_4_xyz}" rpy="${joint_4_rpy}" />
       <parent link="${prefix}forearm_link" />
       <child link="${prefix}lower_wrist_link" />
@@ -375,5 +393,5 @@
     </link>
     <joint name="${prefix}joint_5" type="revolute">
-      <origin xyz="0 -0.062957 -0.22275" rpy="-1.5707963267948966 0 0" />
+      <origin xyz="${joint_5_xyz}" rpy="${joint_5_rpy}" />
       <parent link="${prefix}lower_wrist_link" />
       <child link="${prefix}upper_wrist_link" />
@@ -410,5 +428,5 @@
     </link>
     <joint name="${prefix}joint_6" type="revolute">
-      <origin xyz="0.087028 0.086 -0.076922" rpy="0 -1.5707963267948966 0" />
+      <origin xyz="${joint_6_xyz}" rpy="${joint_6_rpy}" />
       <parent link="${prefix}upper_wrist_link" />
       <child link="${prefix}wrist_interface_link" />

Commit message: Fixed issue when handling the gripper parameter in urdf; fixed issue when checking the number of joints in hardware interface

File: link6_description/urdf/link6.urdf.xacro (robot description, xacro)
@@ -9,5 +9,5 @@
     <xacro:arg name="session_inactivity_timeout_ms" default="60000" />
     <xacro:arg name="connection_inactivity_timeout_ms" default="2000" />
-    <xacro:arg name="gripper" default="$(arg gripper)" />
+    <xacro:arg name="gripper" default="" />
     <xacro:arg name="gripper_joint_name" default="" />
     <xacro:arg name="gripper_b_joint_name" default="" />
@@ -48,6 +48,8 @@
         <origin xyz="0 0 0" rpy="0 0 0" />  <!-- position robot in the world -->
     </xacro:link6>
+    <!-- Conditionally include gripper -->
+    <xacro:property name="gripper" value="$(arg gripper)"/>
     <!-- If no gripper, define tool frame here -->
-    <xacro:if value="${gripper == ''}">
+    <xacro:if value="${not gripper}">
         <link name="$(arg prefix)tool_frame" />
         <joint name="$(arg prefix)tool_frame_joint" type="fixed">
@@ -59,5 +61,5 @@
     </xacro:if>
     <!-- Include and load the gripper if defined -->
-    <xacro:if value="${gripper != ''}">
+    <xacro:unless value="${not gripper}">
         <xacro:include filename="$(find link6_description)/urdf/grippers/$(arg gripper)_macro.xacro" />
         <xacro:load_gripper
@@ -69,5 +71,5 @@
             use_internal_bus_gripper_comm="$(arg use_internal_bus_gripper_comm)">
         </xacro:load_gripper>
-    </xacro:if>
+    </xacro:unless>
     <xacro:if value="$(arg sim_gazebo)">
         <gazebo>
