Commit message: Updates to multiple files to work properly with the real hardware

File: link6_description/urdf/link6.ros2_control.xacro (robot description, xacro)
@@ -133,4 +133,9 @@
         <state_interface name="effort" />
       </joint>
+      <joint name="${prefix}robotiq_85_left_knuckle_joint">
+          <command_interface name="position" />
+          <state_interface name="position"/>
+          <state_interface name="velocity"/>
+      </joint>
     </ros2_control>
   </xacro:macro>

File: link6_description/urdf/link6.urdf.xacro (robot description, xacro)
@@ -26,28 +26,6 @@
     <xacro:property name="initial_positions_file" default="$(arg initial_positions_file)" />
     <link name="world" />
-    <joint name="world_joint" type="fixed">
-        <parent link="world" />
-        <child link="table" />
-        <origin xyz="0 0 1.0" rpy="0 0 0" />
-    </joint>
-    <link name="table">
-        <visual>
-            <origin xyz="0 0 -0.02" rpy="0 0 0" />
-            <geometry>
-                <box size="1.0 1.0 0.04" />
-            </geometry>
-            <material name="white">
-                <color rgba="1 1 1 1.0" />
-            </material>
-        </visual>
-        <collision>
-            <origin xyz="0 0 -0.02" rpy="0 0 0" />
-            <geometry>
-                <box size="1.0 1.0 0.04" />
-            </geometry>
-        </collision>
-    </link>
     <xacro:link6
-        parent="table"
+        parent="world"
         prefix="$(arg prefix)"
         gripper="$(arg gripper)"

File: link6_description/urdf/link6_macro.xacro (robot description, xacro)
@@ -434,5 +434,5 @@
         use_fake_hardware="${use_fake_hardware}"
         fake_sensor_commands="${fake_sensor_commands}"
-        include_ros2_control="true"
+        include_ros2_control="false"
         com_port="${gripper_com_port}"
         sim_ignition="${sim_gazebo}">

Commit message: Added 90 degrees double gripper. Modular approach now working in simulation

File: link6_description/urdf/link6.ros2_control.xacro (robot description, xacro)
@@ -28,17 +28,4 @@
         <xacro:unless value="${use_fake_hardware or sim_gazebo}">
           <xacro:unless value="${moveit_active}">
-            <!-- <plugin>kortex_driver/KortexMultiInterfaceHardware</plugin>
-            <param name="robot_ip">${robot_ip}</param>
-            <param name="username">${username}</param>
-            <param name="password">${password}</param>
-            <param name="port">${port}</param>
-            <param name="port_realtime">${port_realtime}</param>
-            <param name="session_inactivity_timeout_ms">${session_inactivity_timeout_ms}</param>
-            <param name="connection_inactivity_timeout_ms">${connection_inactivity_timeout_ms}</param>
-            <param name="tf_prefix">"${tf_prefix}"</param>
-            <param name="use_internal_bus_gripper_comm">${use_internal_bus_gripper_comm}</param>
-            <param name="gripper_joint_name">${gripper_joint_name}</param>
-            <param name="gripper_max_velocity">${gripper_max_velocity}</param>
-            <param name="gripper_max_force">${gripper_max_force}</param> -->
             <plugin>kortex3_driver/Kortex3HardwareInterface</plugin>
             <param name="robot_ip">${robot_ip}</param>
@@ -48,17 +35,4 @@
         </xacro:unless>
         <xacro:if value="${moveit_active}">
-          <!-- <plugin>kortex_driver/KortexMultiInterfaceHardware</plugin>
-          <param name="robot_ip">${robot_ip}</param>
-          <param name="username">${username}</param>
-          <param name="password">${password}</param>
-          <param name="port">${port}</param>
-          <param name="port_realtime">${port_realtime}</param>
-          <param name="session_inactivity_timeout_ms">${session_inactivity_timeout_ms}</param>
-          <param name="connection_inactivity_timeout_ms">${connection_inactivity_timeout_ms}</param>
-          <param name="tf_prefix">"${tf_prefix}"</param>
-          <param name="use_internal_bus_gripper_comm">${use_internal_bus_gripper_comm}</param>
-          <param name="gripper_joint_name">${gripper_joint_name}</param>
-          <param name="gripper_max_velocity">${gripper_max_velocity}</param>
-          <param name="gripper_max_force">${gripper_max_force}</param> -->
           <plugin>kortex3_driver/Kortex3HardwareInterface</plugin>
           <param name="robot_ip">${robot_ip}</param>
@@ -133,9 +107,11 @@
         <state_interface name="effort" />
       </joint>
-      <joint name="${prefix}robotiq_85_left_knuckle_joint">
+      <xacro:unless value="${sim_gazebo}">
+        <joint name="${prefix}robotiq_85_left_knuckle_joint">
           <command_interface name="position" />
-          <state_interface name="position"/>
-          <state_interface name="velocity"/>
-      </joint>
+          <state_interface name="position" />
+          <state_interface name="velocity" />
+        </joint>
+      </xacro:unless>
     </ros2_control>
   </xacro:macro>

File: link6_description/urdf/link6_macro.xacro (robot description, xacro)
@@ -1,6 +1,5 @@
 <?xml version="1.0" encoding="utf-8"?>
 <robot name="link6" xmlns:xacro="http://www.ros.org/wiki/xacro">
-  <xacro:macro name="link6"
-    params="
+  <xacro:macro name="link6" params="
     parent
     *origin
@@ -17,7 +16,4 @@
     gripper_com_port_right:=/dev/ttyUSB1
     moveit_active:=false">
-    <!-- Available grippers defined here -->
-    <xacro:property name="available_grippers" value="['robotiq_2f_85', 'double_gripper']"/>
-    <xacro:property name="PI" value="3.14159"/>
     <!-- ros2 control include -->
     <xacro:include filename="$(find link6_description)/urdf/link6.ros2_control.xacro" />
@@ -419,20 +415,31 @@
       <child link="${prefix}end_effector_link" />
     </joint>
-    <!-- Include and load gripper logic based off of available grippers for link_6 -->
+    <!-- If no gripper, define tool frame here -->
+    <xacro:if value="${gripper == ''}">
+      <link name="${prefix}tool_frame" />
+      <joint name="${prefix}tool_frame_joint" type="fixed">
+        <origin xyz="0 0 0" rpy="0 0 0" />
+        <parent link="${prefix}end_effector_link" />
+        <child link="${prefix}tool_frame" />
+        <axis xyz="0 0 0" />
+      </joint>
+    </xacro:if>
+    <!-- Include and load gripper based on available grippers for Link6 -->
     <xacro:if value="${gripper == 'robotiq_2f_85'}">
       <xacro:include filename="$(find robotiq_description)/urdf/robotiq_2f_85_macro.urdf.xacro" />
-        <xacro:robotiq_gripper
-          name="robotiq_single_gripper"
-          parent="${prefix}end_effector_link"
-          prefix="${prefix}"
-          use_fake_hardware="${use_fake_hardware}"
-          fake_sensor_commands="${fake_sensor_commands}"
-          com_port="${gripper_com_port_left}"
-          sim_ignition="${sim_gazebo}">
-          <origin xyz="0 0 0.05" rpy="${PI/4} 0 0" />
-        </xacro:robotiq_gripper>
+      <xacro:robotiq_gripper
+        name="RobotiqGripperHardwareInterface"
+        parent="${prefix}end_effector_link"
+        prefix="${prefix}"
+        use_fake_hardware="${use_fake_hardware}"
+        fake_sensor_commands="${fake_sensor_commands}"
+        include_ros2_control="${sim_gazebo}"
+        com_port="${gripper_com_port_left}"
+        sim_ignition="${sim_gazebo}">
+        <origin xyz="0 0 0" rpy="0 0 0" />
+      </xacro:robotiq_gripper>
     </xacro:if>
-    <xacro:if value="${gripper == 'double_gripper'}">
-      <xacro:include filename="$(find agri_harveyl_description)/urdf/double_gripper_macro.urdf.xacro" />
+    <xacro:if value="${gripper == 'double_robotiq'}">
+      <xacro:include filename="$(find link6_description)/urdf/double_robotiq_macro.urdf.xacro" />
       <xacro:double_robotiq_gripper
         parent="${prefix}end_effector_link"
@@ -446,13 +453,16 @@
       </xacro:double_robotiq_gripper>
     </xacro:if>
-    <!-- If no gripper, define tool frame here -->
-    <xacro:if value="${gripper == ''}">
-      <link name="${prefix}tool_frame" />
-      <joint name="${prefix}tool_frame_joint" type="fixed">
-        <origin xyz="0 0 0" rpy="0 0 0" />
-        <parent link="${prefix}end_effector_link" />
-        <child link="${prefix}tool_frame" />
-        <axis xyz="0 0 0" />
-      </joint>
+    <xacro:if value="${gripper == 'double_robotiq_90'}">
+      <xacro:include filename="$(find link6_description)/urdf/double_robotiq_90_macro.urdf.xacro" />
+      <xacro:double_robotiq_gripper_90
+        parent="${prefix}end_effector_link"
+        prefix="${prefix}"
+        use_fake_hardware="${use_fake_hardware}"
+        fake_sensor_commands="${fake_sensor_commands}"
+        use_sim="${sim_gazebo}"
+        com_port_left="${gripper_com_port_left}"
+        com_port_right="${gripper_com_port_right}">
+        <origin xyz="0 0 0" rpy="0 0 0" />
+      </xacro:double_robotiq_gripper_90>
     </xacro:if>
   </xacro:macro>

Commit message: Added a second gripper interface to allow sending commands to both grippers at the same time

File: link6_description/urdf/link6.ros2_control.xacro (robot description, xacro)
@@ -11,4 +11,5 @@
     username
     password
+    gripper_modbus_id:=9
     moveit_active:=false">
     <ros2_control name="${prefix}Kortex3Interface" type="system">
@@ -32,4 +33,5 @@
             <param name="username">${username}</param>
             <param name="password">${password}</param>
+            <param name="gripper_modbus_id">${gripper_modbus_id}</param>
           </xacro:unless>
         </xacro:unless>
@@ -39,4 +41,5 @@
           <param name="username">${username}</param>
           <param name="password">${password}</param>
+          <param name="gripper_modbus_id">${gripper_modbus_id}</param>
         </xacro:if>
       </hardware>
@@ -108,5 +111,10 @@
       </joint>
       <xacro:unless value="${sim_gazebo}">
-        <joint name="${prefix}robotiq_85_left_knuckle_joint">
+        <joint name="${prefix}right_robotiq_85_left_knuckle_joint">
+          <command_interface name="position" />
+          <state_interface name="position" />
+          <state_interface name="velocity" />
+        </joint>
+        <joint name="${prefix}left_robotiq_85_left_knuckle_joint">
           <command_interface name="position" />
           <state_interface name="position" />

Commit message: Updated gripper pose calculation and ros2_control joints to work properly with the Robotiq Hande

File: link6_description/urdf/link6.ros2_control.xacro (robot description, xacro)
@@ -125,4 +125,9 @@
             <state_interface name="velocity" />
           </joint>
+          <joint name="${prefix}left_robotiq_hande_left_finger_joint">
+            <command_interface name="position" />
+            <state_interface name="position" />
+            <state_interface name="velocity" />
+          </joint>
         </xacro:if>
         <xacro:if value="${gripper == 'double_robotiq_90'}">

Commit message: Temporary workaround to avoid warnings

File: link6_description/urdf/link6.ros2_control.xacro (robot description, xacro)
@@ -125,5 +125,5 @@
             <state_interface name="velocity" />
           </joint>
-          <joint name="${prefix}left_robotiq_hande_left_finger_joint">
+          <joint name="${prefix}robotiq_hande_left_finger_joint">
             <command_interface name="position" />
             <state_interface name="position" />

Commit message: Added condition to load joint in urdf, removed unused config file, readded controllers to sim launch file

File: link6_description/urdf/link6.ros2_control.xacro (robot description, xacro)
@@ -133,9 +133,11 @@
         <state_interface name="effort" />
       </joint>
-      <joint name="${prefix}robotiq_85_left_knuckle_joint">
-          <command_interface name="position" />
-          <state_interface name="position"/>
-          <state_interface name="velocity"/>
-      </joint>
+      <xacro:unless value="${sim_gazebo}">
+        <joint name="${prefix}robotiq_85_left_knuckle_joint">
+            <command_interface name="position" />
+            <state_interface name="position"/>
+            <state_interface name="velocity"/>
+        </joint>
+      </xacro:unless>
     </ros2_control>
   </xacro:macro>

Commit message: Added possibility to load different grippers; added a second gripper joint name to urdf to enable controlling two grippers

File: link6_description/urdf/link6.ros2_control.xacro (robot description, xacro)
@@ -4,13 +4,16 @@
     params="
     prefix
+    robot_ip
+    username:=admin
+    password:=admin
+    use_internal_bus_gripper_comm:=false
     gripper
+    gripper_joint_name
+    gripper_b_joint_name
+    gripper_modbus_id:=9
     use_fake_hardware:=false
     fake_sensor_commands:=false
     sim_gazebo:=false
     initial_positions:=${dict(joint_1=0.0,joint_2=0.0,joint_3=0.0,joint_4=0.0,joint_5=0.0,joint_6=0.0)}
-    robot_ip
-    username
-    password
-    gripper_modbus_id:=9
     moveit_active:=false">
     <ros2_control name="${prefix}Kortex3Interface" type="system">
@@ -35,4 +38,6 @@
             <param name="password">${password}</param>
             <param name="gripper">${gripper}</param>
+            <param name="gripper_joint_name">${gripper_joint_name}</param>
+            <param name="gripper_b_joint_name">${gripper_b_joint_name}</param>
             <param name="gripper_modbus_id">${gripper_modbus_id}</param>
           </xacro:unless>
@@ -44,4 +49,6 @@
           <param name="password">${password}</param>
           <param name="gripper">${gripper}</param>
+          <param name="gripper_joint_name">${gripper_joint_name}</param>
+          <param name="gripper_b_joint_name">${gripper_b_joint_name}</param>
           <param name="gripper_modbus_id">${gripper_modbus_id}</param>
         </xacro:if>
@@ -113,36 +120,20 @@
         <state_interface name="effort" />
       </joint>
-      <xacro:unless value="${sim_gazebo}">
-        <xacro:if value="${gripper == 'robotiq_2f_85'}">
-          <joint name="${prefix}robotiq_85_left_knuckle_joint">
-            <command_interface name="position" />
-            <state_interface name="position" />
-            <state_interface name="velocity" />
-          </joint>
-        </xacro:if>
-        <xacro:if value="${gripper == 'robotiq_hande'}">
-          <joint name="${prefix}robotiq_hande_left_finger_joint">
-            <command_interface name="position" />
-            <state_interface name="position" />
-            <state_interface name="velocity" />
-          </joint>
-          <joint name="${prefix}robotiq_hande_left_finger_joint">
-            <command_interface name="position" />
-            <state_interface name="position" />
-            <state_interface name="velocity" />
-          </joint>
-        </xacro:if>
-        <xacro:if value="${gripper == 'double_robotiq_90'}">
-          <joint name="${prefix}right_robotiq_hande_left_finger_joint">
-            <command_interface name="position" />
-            <state_interface name="position" />
-            <state_interface name="velocity" />
-          </joint>
-          <joint name="${prefix}left_robotiq_hande_left_finger_joint">
-            <command_interface name="position" />
-            <state_interface name="position" />
-            <state_interface name="velocity" />
-          </joint>
-        </xacro:if>
+      <!-- If using the real robot, we need to define gripper joints for the hardware interface -->
+      <xacro:unless value="${use_fake_hardware or sim_gazebo}">
+        <xacro:unless value="${not gripper}">
+          <xacro:if value="${use_internal_bus_gripper_comm}">
+            <joint name="${prefix}${gripper_joint_name}">
+              <command_interface name="position" />
+              <state_interface name="position"/>
+              <state_interface name="velocity"/>
+            </joint>
+            <joint name="${prefix}${gripper_b_joint_name}">
+              <command_interface name="position" />
+              <state_interface name="position"/>
+              <state_interface name="velocity"/>
+            </joint>
+          </xacro:if>
+        </xacro:unless>
       </xacro:unless>
     </ros2_control>

File: link6_description/urdf/link6.urdf.xacro (robot description, xacro)
@@ -11,4 +11,5 @@
     <xacro:arg name="gripper" default="" />
     <xacro:arg name="gripper_joint_name" default="finger_joint" />
+    <xacro:arg name="gripper_b_joint_name" default="finger_joint_2" />
     <xacro:arg name="gripper_max_velocity" default="100.0" />
     <xacro:arg name="gripper_max_force" default="100.0" />
@@ -19,4 +20,5 @@
     <xacro:arg name="use_internal_bus_gripper_comm" default="false" />
     <xacro:arg name="use_external_cable" default="false" />
+    <xacro:property name="gripper" value="$(arg gripper)"/>
     <xacro:include filename="$(find link6_description)/urdf/link6_macro.xacro" />
     <!-- initial position for simulations (Mock Hardware, Gazebo) -->
@@ -29,8 +31,11 @@
         parent="world"
         prefix="$(arg prefix)"
-        gripper="$(arg gripper)"
         robot_ip="$(arg robot_ip)"
         username="$(arg username)"
         password="$(arg password)"
+        use_internal_bus_gripper_comm="$(arg use_internal_bus_gripper_comm)"
+        gripper="$(arg gripper)"
+        gripper_joint_name="$(arg gripper_joint_name)"
+        gripper_b_joint_name="$(arg gripper_b_joint_name)"
         use_fake_hardware="$(arg use_fake_hardware)"
         fake_sensor_commands="$(arg fake_sensor_commands)"
@@ -39,11 +44,26 @@
         <origin xyz="0 0 0" rpy="0 0 0" />  <!-- position robot in the world -->
     </xacro:link6>
-    <link name="$(arg prefix)tool_frame" />
-    <joint name="$(arg prefix)tool_frame_joint" type="fixed">
-        <origin xyz="0 0 0" rpy="0 0 0" />
-        <parent link="$(arg prefix)end_effector_link" />
-        <child link="$(arg prefix)tool_frame" />
-        <axis xyz="0 0 0" />
-    </joint>
+    <!-- If no gripper, define tool frame here -->
+    <xacro:if value="${gripper == ''}">
+        <link name="$(arg prefix)tool_frame" />
+        <joint name="$(arg prefix)tool_frame_joint" type="fixed">
+            <origin xyz="0 0 0" rpy="0 0 0" />
+            <parent link="$(arg prefix)end_effector_link" />
+            <child link="$(arg prefix)tool_frame" />
+            <axis xyz="0 0 0" />
+        </joint>
+    </xacro:if>
+    <!-- Include and load the gripper if defined -->
+    <xacro:if value="${gripper != ''}">
+        <xacro:include filename="$(find link6_description)/urdf/grippers/$(arg gripper)_macro.xacro" />
+        <xacro:load_gripper
+            prefix="$(arg prefix)"
+            parent="$(arg prefix)end_effector_link"
+            sim_gazebo="$(arg sim_gazebo)"
+            use_fake_hardware="$(arg use_fake_hardware)"
+            fake_sensor_commands="$(arg fake_sensor_commands)"
+            use_internal_bus_gripper_comm="$(arg use_internal_bus_gripper_comm)">
+        </xacro:load_gripper>
+    </xacro:if>
     <xacro:if value="$(arg sim_gazebo)">
         <gazebo>

File: link6_description/urdf/link6_macro.xacro (robot description, xacro)
@@ -5,14 +5,15 @@
     *origin
     prefix:=''
-    gripper
     robot_ip
     username:=admin
     password:=admin
+    use_internal_bus_gripper_comm:=false
+    gripper
+    gripper_joint_name:='finger_joint'
+    gripper_b_joint_name:='finger_joint_2'
     use_fake_hardware:=false
     fake_sensor_commands:=false
     sim_gazebo:=false
     initial_positions:=${dict(joint_1=0.0,joint_2=0.0,joint_3=0.0,joint_4=0.0,joint_5=0.0,joint_6=0.0)}
-    gripper_com_port_left:=/dev/ttyUSB0
-    gripper_com_port_right:=/dev/ttyUSB1
     moveit_active:=false">
     <!-- Properties -->
@@ -28,12 +29,15 @@
     <xacro:link6_ros2_control
       prefix="${prefix}"
+      robot_ip="${robot_ip}"
+      username="${username}"
+      password="${password}"
+      use_internal_bus_gripper_comm="${use_internal_bus_gripper_comm}"
       gripper="${gripper}"
+      gripper_joint_name="${gripper_joint_name}"
+      gripper_b_joint_name="${gripper_b_joint_name}"
       use_fake_hardware="${use_fake_hardware}"
       fake_sensor_commands="${fake_sensor_commands}"
       sim_gazebo="${sim_gazebo}"
       initial_positions="${initial_positions}"
-      robot_ip="${robot_ip}"
-      username="${username}"
-      password="${password}"
       moveit_active="${moveit_active}" />
     <!-- Define material colors -->
