Commit message: Wrapped all gripper related objects and variables in a class; hardware interface creates and manages two grippers

File: link6_description/urdf/link6.ros2_control.xacro (robot description, xacro)
@@ -9,7 +9,8 @@
     use_internal_bus_gripper_comm:=false
     gripper
-    gripper_joint_name
-    gripper_b_joint_name
+    gripper_joint_name:=''
+    gripper_b_joint_name:=''
     gripper_modbus_id:=9
+    gripper_b_modbus_id:=10
     use_fake_hardware:=false
     fake_sensor_commands:=false
@@ -42,4 +43,5 @@
             <param name="gripper_b_joint_name">${gripper_b_joint_name}</param>
             <param name="gripper_modbus_id">${gripper_modbus_id}</param>
+            <param name="gripper_b_modbus_id">${gripper_b_modbus_id}</param>
           </xacro:unless>
         </xacro:unless>
@@ -54,4 +56,5 @@
           <param name="gripper_b_joint_name">${gripper_b_joint_name}</param>
           <param name="gripper_modbus_id">${gripper_modbus_id}</param>
+          <param name="gripper_b_modbus_id">${gripper_b_modbus_id}</param>
         </xacro:if>
       </hardware>
@@ -126,14 +129,20 @@
         <xacro:unless value="${not gripper}">
           <xacro:if value="${use_internal_bus_gripper_comm}">
-            <joint name="${prefix}${gripper_joint_name}">
-              <command_interface name="position" />
-              <state_interface name="position"/>
-              <state_interface name="velocity"/>
-            </joint>
-            <joint name="${prefix}${gripper_b_joint_name}">
-              <command_interface name="position" />
-              <state_interface name="position"/>
-              <state_interface name="velocity"/>
-            </joint>
+            <!-- Gripper A joint (only if gripper_joint_name is defined and not empty) -->
+            <xacro:unless value="${gripper_joint_name == '' or gripper_joint_name == None}">
+              <joint name="${prefix}${gripper_joint_name}">
+                <command_interface name="position" />
+                <state_interface name="position"/>
+                <state_interface name="velocity"/>
+              </joint>
+            </xacro:unless>
+            <!-- Gripper B joint (only if gripper_b_joint_name is defined and not empty) -->
+            <xacro:unless value="${gripper_b_joint_name == '' or gripper_b_joint_name == None}">
+              <joint name="${prefix}${gripper_b_joint_name}">
+                <command_interface name="position" />
+                <state_interface name="position"/>
+                <state_interface name="velocity"/>
+              </joint>
+            </xacro:unless>
           </xacro:if>
         </xacro:unless>

File: link6_description/urdf/link6.urdf.xacro (robot description, xacro)
@@ -11,5 +11,5 @@
     <xacro:arg name="gripper" default="" />
     <xacro:arg name="gripper_joint_name" default="finger_joint" />
-    <xacro:arg name="gripper_b_joint_name" default="finger_joint_2" />
+    <xacro:arg name="gripper_b_joint_name" default="" />
     <xacro:arg name="gripper_max_velocity" default="100.0" />
     <xacro:arg name="gripper_max_force" default="100.0" />

File: link6_description/urdf/link6_macro.xacro (robot description, xacro)
@@ -10,6 +10,6 @@
     use_internal_bus_gripper_comm:=false
     gripper
-    gripper_joint_name:='finger_joint'
-    gripper_b_joint_name:='finger_joint_2'
+    gripper_joint_name:=''
+    gripper_b_joint_name:=''
     use_fake_hardware:=false
     fake_sensor_commands:=false

Commit message: Changed the hardware interface to send low level position commands instead of high level velocity commands

File: link6_description/urdf/link6.ros2_control.xacro (robot description, xacro)
@@ -64,4 +64,8 @@
           <param name="max">3.14</param>
         </command_interface>
+        <command_interface name="position">
+          <param name="min">-3.14</param>
+          <param name="max">3.14</param>
+        </command_interface>
         <state_interface name="position">
           <param name="initial_value">${initial_positions['joint_1']}</param>
@@ -72,4 +76,8 @@
       <joint name="${prefix}joint_2">
         <command_interface name="velocity">
+          <param name="min">-3.14</param>
+          <param name="max">3.14</param>
+        </command_interface>
+        <command_interface name="position">
           <param name="min">-3.14</param>
           <param name="max">3.14</param>
@@ -86,4 +94,8 @@
           <param name="max">3.14</param>
         </command_interface>
+        <command_interface name="position">
+          <param name="min">-3.14</param>
+          <param name="max">3.14</param>
+        </command_interface>
         <state_interface name="position">
           <param name="initial_value">${initial_positions['joint_3']}</param>
@@ -94,4 +106,8 @@
       <joint name="${prefix}joint_4">
         <command_interface name="velocity">
+          <param name="min">-6.28</param>
+          <param name="max">6.28</param>
+        </command_interface>
+        <command_interface name="position">
           <param name="min">-6.28</param>
           <param name="max">6.28</param>
@@ -108,4 +124,8 @@
           <param name="max">6.28</param>
         </command_interface>
+        <command_interface name="position">
+          <param name="min">-6.28</param>
+          <param name="max">6.28</param>
+        </command_interface>
         <state_interface name="position">
           <param name="initial_value">${initial_positions['joint_5']}</param>
@@ -116,4 +136,8 @@
       <joint name="${prefix}joint_6">
         <command_interface name="velocity">
+          <param name="min">-6.28</param>
+          <param name="max">6.28</param>
+        </command_interface>
+        <command_interface name="position">
           <param name="min">-6.28</param>
           <param name="max">6.28</param>

File: link6_description/urdf/link6_macro.xacro (robot description, xacro)
@@ -150,5 +150,7 @@
       <child link="${prefix}shoulder_link" />
       <axis xyz="0 0 1" />
-      <limit lower="-6.283185307179586" upper="6.283185307179586" effort="210"
+      <!-- <limit lower="-6.283185307179586" upper="6.283185307179586" effort="210"
+        velocity="3.141592653589793" /> -->
+      <limit lower="-6.283185307179586" upper="0.0" effort="210"
         velocity="3.141592653589793" />
     </joint>
@@ -239,5 +241,7 @@
       <child link="${prefix}arm_link" />
       <axis xyz="0 0 1" />
-      <limit lower="-6.283185307179586" upper="6.283185307179586" effort="210"
+      <!-- <limit lower="-6.283185307179586" upper="6.283185307179586" effort="210"
+        velocity="3.141592653589793" /> -->
+      <limit lower="-0.5236" upper="1.3963" effort="210"
         velocity="3.141592653589793" />
     </joint>
@@ -292,7 +296,9 @@
       <child link="${prefix}forearm_link" />
       <axis xyz="0 0 1" />
-      <limit lower="-6.283185307179586" upper="6.283185307179586" effort="210"
+      <!-- <limit lower="-6.283185307179586" upper="6.283185307179586" effort="210"
+        velocity="3.141592653589793" /> -->
+      <limit lower="-2.7925" upper="0.0" effort="210"
         velocity="3.141592653589793" />
-      <initial_position>1.57079632679</initial_position>
+      <!-- <initial_position>1.57079632679</initial_position> -->
     </joint>
     <link name="${prefix}lower_wrist_link">
@@ -352,5 +358,7 @@
       <child link="${prefix}lower_wrist_link" />
       <axis xyz="0 0 1" />
-      <limit lower="-6.283185307179586" upper="6.283185307179586" effort="100"
+      <!-- <limit lower="-6.283185307179586" upper="6.283185307179586" effort="100"
+        velocity="6.283185307179586" /> -->
+      <limit lower="-3.5" upper="-2.5" effort="100"
         velocity="6.283185307179586" />
     </joint>
@@ -406,5 +414,7 @@
       <child link="${prefix}upper_wrist_link" />
       <axis xyz="0 0 1" />
-      <limit lower="-6.283185307179586" upper="6.283185307179586" effort="100"
+      <!-- <limit lower="-6.283185307179586" upper="6.283185307179586" effort="100"
+        velocity="6.283185307179586" /> -->
+      <limit lower="-0.3" upper="1.8" effort="100"
         velocity="6.283185307179586" />
     </joint>
@@ -441,5 +451,7 @@
       <child link="${prefix}wrist_interface_link" />
       <axis xyz="0 0 1" />
-      <limit lower="-6.283185307179586" upper="6.283185307179586" effort="100"
+      <!-- <limit lower="-6.283185307179586" upper="6.283185307179586" effort="100"
+        velocity="6.283185307179586" /> -->
+      <limit lower="-1.9" upper="3.2" effort="100"
         velocity="6.283185307179586" />
     </joint>
