Commit message: Modified URDF to allow selecting between high-level or low-level mode. Added new bringup launch file and controller parameters file. Added twist controller

File: link6_description/urdf/link6.ros2_control.xacro (robot description, xacro)
@@ -20,22 +20,34 @@
     fake_sensor_commands:=false
     sim_gazebo:=false
-    initial_positions:=${dict(joint_1=0.0,joint_2=0.0,joint_3=0.0,joint_4=0.0,joint_5=0.0,joint_6=0.0)}
-    moveit_active:=false">
+    low_level_mode:=false
+    initial_positions:=${dict(joint_1=0.0,joint_2=0.0,joint_3=0.0,joint_4=0.0,joint_5=0.0,joint_6=0.0)}">
     <ros2_control name="${prefix}Kortex3Interface" type="system">
       <hardware>
         <xacro:if value="${sim_gazebo}">
-          <xacro:unless value="${moveit_active}">
-            <plugin>gz_ros2_control/GazeboSimSystem</plugin>
-          </xacro:unless>
+          <plugin>gz_ros2_control/GazeboSimSystem</plugin>
         </xacro:if>
         <xacro:if value="${use_fake_hardware}">
-          <xacro:unless value="${moveit_active}">
-            <plugin>mock_components/GenericSystem</plugin>
-            <param name="fake_sensor_commands">${fake_sensor_commands}</param>
-            <param name="state_following_offset">0.0</param>
-          </xacro:unless>
+          <plugin>mock_components/GenericSystem</plugin>
+          <param name="fake_sensor_commands">${fake_sensor_commands}</param>
+          <param name="state_following_offset">0.0</param>
         </xacro:if>
         <xacro:unless value="${use_fake_hardware or sim_gazebo}">
-          <xacro:unless value="${moveit_active}">
+          <xacro:unless value="${low_level_mode}">
+            <plugin>kortex3_driver/Kortex3HardwareInterface</plugin>
+            <param name="robot_ip">${robot_ip}</param>
+            <param name="username">${username}</param>
+            <param name="password">${password}</param>
+            <param name="port">${port}</param>
+            <param name="port_realtime">${port_realtime}</param>
+            <param name="session_inactivity_timeout_ms">${session_inactivity_timeout_ms}</param>
+            <param name="connection_inactivity_timeout_ms">${connection_inactivity_timeout_ms}</param>
+            <param name="use_internal_bus_gripper_comm">${use_internal_bus_gripper_comm}</param>
+            <param name="gripper">${gripper}</param>
+            <param name="gripper_joint_name">${prefix}${gripper_joint_name}</param>
+            <param name="gripper_b_joint_name">${prefix}${gripper_b_joint_name}</param>
+            <param name="gripper_modbus_id">${gripper_modbus_id}</param>
+            <param name="gripper_b_modbus_id">${gripper_b_modbus_id}</param>
+          </xacro:unless>
+          <xacro:if value="${low_level_mode}">
             <plugin>kortex3_driver/KortexHardwareInterface</plugin>
             <param name="robot_ip">${robot_ip}</param>
@@ -52,136 +64,190 @@
             <param name="gripper_modbus_id">${gripper_modbus_id}</param>
             <param name="gripper_b_modbus_id">${gripper_b_modbus_id}</param>
+          </xacro:if>
+        </xacro:unless>
+      </hardware>
+      <xacro:unless value="${low_level_mode}">
+        <joint name="${prefix}joint_1">
+          <command_interface name="velocity">
+            <param name="min">-3.14</param>
+            <param name="max">3.14</param>
+          </command_interface>
+          <state_interface name="position">
+            <param name="initial_value">${initial_positions['joint_1']}</param>
+          </state_interface>
+          <state_interface name="velocity" />
+          <state_interface name="effort" />
+        </joint>
+        <joint name="${prefix}joint_2">
+          <command_interface name="velocity">
+            <param name="min">-3.14</param>
+            <param name="max">3.14</param>
+          </command_interface>
+          <state_interface name="position">
+            <param name="initial_value">${initial_positions['joint_2']}</param>
+          </state_interface>
+          <state_interface name="velocity" />
+          <state_interface name="effort" />
+        </joint>
+        <joint name="${prefix}joint_3">
+          <command_interface name="velocity">
+            <param name="min">-3.14</param>
+            <param name="max">3.14</param>
+          </command_interface>
+          <state_interface name="position">
+            <param name="initial_value">${initial_positions['joint_3']}</param>
+          </state_interface>
+          <state_interface name="velocity" />
+          <state_interface name="effort" />
+        </joint>
+        <joint name="${prefix}joint_4">
+          <command_interface name="velocity">
+            <param name="min">-6.28</param>
+            <param name="max">6.28</param>
+          </command_interface>
+          <state_interface name="position">
+            <param name="initial_value">${initial_positions['joint_4']}</param>
+          </state_interface>
+          <state_interface name="velocity" />
+          <state_interface name="effort" />
+        </joint>
+        <joint name="${prefix}joint_5">
+          <command_interface name="velocity">
+            <param name="min">-6.28</param>
+            <param name="max">6.28</param>
+          </command_interface>
+          <state_interface name="position">
+            <param name="initial_value">${initial_positions['joint_5']}</param>
+          </state_interface>
+          <state_interface name="velocity" />
+          <state_interface name="effort" />
+        </joint>
+        <joint name="${prefix}joint_6">
+          <command_interface name="velocity">
+            <param name="min">-6.28</param>
+            <param name="max">6.28</param>
+          </command_interface>
+          <state_interface name="position">
+            <param name="initial_value">${initial_positions['joint_6']}</param>
+          </state_interface>
+          <state_interface name="velocity" />
+          <state_interface name="effort" />
+        </joint>
+        <!-- If using the real robot, we need to define gripper joints for the hardware interface -->
+        <xacro:unless value="${use_fake_hardware or sim_gazebo}">
+          <xacro:unless value="${not gripper}">
+            <xacro:if value="${use_internal_bus_gripper_comm}">
+              <!-- Gripper A joint (only if gripper_joint_name is defined and not empty) -->
+              <xacro:unless value="${gripper_joint_name == '' or gripper_joint_name == None}">
+                <joint name="${prefix}${gripper_joint_name}">
+                  <command_interface name="position" />
+                  <state_interface name="position"/>
+                  <state_interface name="velocity"/>
+                </joint>
+              </xacro:unless>
+              <!-- Gripper B joint (only if gripper_b_joint_name is defined and not empty) -->
+              <xacro:unless value="${gripper_b_joint_name == '' or gripper_b_joint_name == None}">
+                <joint name="${prefix}${gripper_b_joint_name}">
+                  <command_interface name="position" />
+                  <state_interface name="position"/>
+                  <state_interface name="velocity"/>
+                </joint>
+              </xacro:unless>
+            </xacro:if>
           </xacro:unless>
         </xacro:unless>
-        <xacro:if value="${moveit_active}">
-          <plugin>kortex3_driver/KortexHardwareInterface</plugin>
-          <param name="robot_ip">${robot_ip}</param>
-          <param name="username">${username}</param>
-          <param name="password">${password}</param>
-          <param name="port">${port}</param>
-          <param name="port_realtime">${port_realtime}</param>
-          <param name="session_inactivity_timeout_ms">${session_inactivity_timeout_ms}</param>
-          <param name="connection_inactivity_timeout_ms">${connection_inactivity_timeout_ms}</param>
-          <param name="use_internal_bus_gripper_comm">${use_internal_bus_gripper_comm}</param>
-          <param name="gripper">${gripper}</param>
-          <param name="gripper_joint_name">${prefix}${gripper_joint_name}</param>
-          <param name="gripper_b_joint_name">${prefix}${gripper_b_joint_name}</param>
-          <param name="gripper_modbus_id">${gripper_modbus_id}</param>
-          <param name="gripper_b_modbus_id">${gripper_b_modbus_id}</param>
-        </xacro:if>
-      </hardware>
-      <joint name="${prefix}joint_1">
-        <command_interface name="velocity">
-          <param name="min">-3.14</param>
-          <param name="max">3.14</param>
-        </command_interface>
-        <command_interface name="position">
-          <param name="min">-3.14</param>
-          <param name="max">3.14</param>
-        </command_interface>
-        <state_interface name="position">
-          <param name="initial_value">${initial_positions['joint_1']}</param>
-        </state_interface>
-        <state_interface name="velocity" />
-        <state_interface name="effort" />
-      </joint>
-      <joint name="${prefix}joint_2">
-        <command_interface name="velocity">
-          <param name="min">-3.14</param>
-          <param name="max">3.14</param>
-        </command_interface>
-        <command_interface name="position">
-          <param name="min">-3.14</param>
-          <param name="max">3.14</param>
-        </command_interface>
-        <state_interface name="position">
-          <param name="initial_value">${initial_positions['joint_2']}</param>
-        </state_interface>
-        <state_interface name="velocity" />
-        <state_interface name="effort" />
-      </joint>
-      <joint name="${prefix}joint_3">
-        <command_interface name="velocity">
-          <param name="min">-3.14</param>
-          <param name="max">3.14</param>
-        </command_interface>
-        <command_interface name="position">
-          <param name="min">-3.14</param>
-          <param name="max">3.14</param>
-        </command_interface>
-        <state_interface name="position">
-          <param name="initial_value">${initial_positions['joint_3']}</param>
-        </state_interface>
-        <state_interface name="velocity" />
-        <state_interface name="effort" />
-      </joint>
-      <joint name="${prefix}joint_4">
-        <command_interface name="velocity">
-          <param name="min">-6.28</param>
-          <param name="max">6.28</param>
-        </command_interface>
-        <command_interface name="position">
-          <param name="min">-6.28</param>
-          <param name="max">6.28</param>
-        </command_interface>
-        <state_interface name="position">
-          <param name="initial_value">${initial_positions['joint_4']}</param>
-        </state_interface>
-        <state_interface name="velocity" />
-        <state_interface name="effort" />
-      </joint>
-      <joint name="${prefix}joint_5">
-        <command_interface name="velocity">
-          <param name="min">-6.28</param>
-          <param name="max">6.28</param>
-        </command_interface>
-        <command_interface name="position">
-          <param name="min">-6.28</param>
-          <param name="max">6.28</param>
-        </command_interface>
-        <state_interface name="position">
-          <param name="initial_value">${initial_positions['joint_5']}</param>
-        </state_interface>
-        <state_interface name="velocity" />
-        <state_interface name="effort" />
-      </joint>
-      <joint name="${prefix}joint_6">
-        <command_interface name="velocity">
-          <param name="min">-6.28</param>
-          <param name="max">6.28</param>
-        </command_interface>
-        <command_interface name="position">
-          <param name="min">-6.28</param>
-          <param name="max">6.28</param>
-        </command_interface>
-        <state_interface name="position">
-          <param name="initial_value">${initial_positions['joint_6']}</param>
-        </state_interface>
-        <state_interface name="velocity" />
-        <state_interface name="effort" />
-      </joint>
-      <!-- If using the real robot, we need to define gripper joints for the hardware interface -->
-      <xacro:unless value="${use_fake_hardware or sim_gazebo}">
-        <xacro:unless value="${not gripper}">
-          <xacro:if value="${use_internal_bus_gripper_comm}">
-            <!-- Gripper A joint (only if gripper_joint_name is defined and not empty) -->
-            <!-- <xacro:unless value="${gripper_joint_name == '' or gripper_joint_name == None}">
-              <joint name="${prefix}${gripper_joint_name}">
-                <command_interface name="position" />
-                <state_interface name="position"/>
-                <state_interface name="velocity"/>
-              </joint>
-            </xacro:unless> -->
-            <!-- Gripper B joint (only if gripper_b_joint_name is defined and not empty) -->
-            <!-- <xacro:unless value="${gripper_b_joint_name == '' or gripper_b_joint_name == None}">
-              <joint name="${prefix}${gripper_b_joint_name}">
-                <command_interface name="position" />
-                <state_interface name="position"/>
-                <state_interface name="velocity"/>
-              </joint>
-            </xacro:unless> -->
-          </xacro:if>
-        </xacro:unless>
       </xacro:unless>
+      <xacro:if value="${low_level_mode}">
+        <joint name="${prefix}joint_1">
+          <command_interface name="velocity">
+            <param name="min">-3.14</param>
+            <param name="max">3.14</param>
+          </command_interface>
+          <command_interface name="position">
+            <param name="min">-3.14</param>
+            <param name="max">3.14</param>
+          </command_interface>
+          <state_interface name="position">
+            <param name="initial_value">${initial_positions['joint_1']}</param>
+          </state_interface>
+          <state_interface name="velocity" />
+          <state_interface name="effort" />
+        </joint>
+        <joint name="${prefix}joint_2">
+          <command_interface name="velocity">
+            <param name="min">-3.14</param>
+            <param name="max">3.14</param>
+          </command_interface>
+          <command_interface name="position">
+            <param name="min">-3.14</param>
+            <param name="max">3.14</param>
+          </command_interface>
+          <state_interface name="position">
+            <param name="initial_value">${initial_positions['joint_2']}</param>
+          </state_interface>
+          <state_interface name="velocity" />
+          <state_interface name="effort" />
+        </joint>
+        <joint name="${prefix}joint_3">
+          <command_interface name="velocity">
+            <param name="min">-3.14</param>
+            <param name="max">3.14</param>
+          </command_interface>
+          <command_interface name="position">
+            <param name="min">-3.14</param>
+            <param name="max">3.14</param>
+          </command_interface>
+          <state_interface name="position">
+            <param name="initial_value">${initial_positions['joint_3']}</param>
+          </state_interface>
+          <state_interface name="velocity" />
+          <state_interface name="effort" />
+        </joint>
+        <joint name="${prefix}joint_4">
+          <command_interface name="velocity">
+            <param name="min">-6.28</param>
+            <param name="max">6.28</param>
+          </command_interface>
+          <command_interface name="position">
+            <param name="min">-6.28</param>
+            <param name="max">6.28</param>
+          </command_interface>
+          <state_interface name="position">
+            <param name="initial_value">${initial_positions['joint_4']}</param>
+          </state_interface>
+          <state_interface name="velocity" />
+          <state_interface name="effort" />
+        </joint>
+        <joint name="${prefix}joint_5">
+          <command_interface name="velocity">
+            <param name="min">-6.28</param>
+            <param name="max">6.28</param>
+          </command_interface>
+          <command_interface name="position">
+            <param name="min">-6.28</param>
+            <param name="max">6.28</param>
+          </command_interface>
+          <state_interface name="position">
+            <param name="initial_value">${initial_positions['joint_5']}</param>
+          </state_interface>
+          <state_interface name="velocity" />
+          <state_interface name="effort" />
+        </joint>
+        <joint name="${prefix}joint_6">
+          <command_interface name="velocity">
+            <param name="min">-6.28</param>
+            <param name="max">6.28</param>
+          </command_interface>
+          <command_interface name="position">
+            <param name="min">-6.28</param>
+            <param name="max">6.28</param>
+          </command_interface>
+          <state_interface name="position">
+            <param name="initial_value">${initial_positions['joint_6']}</param>
+          </state_interface>
+          <state_interface name="velocity" />
+          <state_interface name="effort" />
+        </joint>
+      </xacro:if>
     </ros2_control>
   </xacro:macro>

File: link6_description/urdf/link6.urdf.xacro (robot description, xacro)
@@ -22,4 +22,5 @@
     <xacro:arg name="use_internal_bus_gripper_comm" default="false" />
     <xacro:arg name="use_external_cable" default="false" />
+    <xacro:arg name="low_level_mode" default="false" />
     <!-- Initial position for simulations (Mock Hardware, Gazebo) -->
     <xacro:arg name="initial_positions_file" default="$(find link6_description)/config/initial_positions.yaml" />
@@ -48,4 +49,5 @@
         fake_sensor_commands="$(arg fake_sensor_commands)"
         sim_gazebo="$(arg sim_gazebo)"
+        low_level_mode="$(arg low_level_mode)"
         initial_positions_file="$(arg initial_positions_file)"
         calibration_file="$(arg calibration_file)">

File: link6_description/urdf/link6_macro.xacro (robot description, xacro)
@@ -21,5 +21,5 @@
     fake_sensor_commands:=false
     sim_gazebo:=false
-    moveit_active:=false
+    low_level_mode:=false
     initial_positions_file:='$(find link6_description)/config/initial_positions.yaml'
     calibration_file:='$(find link6_description)/config/default_calibration.yaml'">
@@ -69,6 +69,6 @@
       fake_sensor_commands="${fake_sensor_commands}"
       sim_gazebo="${sim_gazebo}"
-      initial_positions="${initial_positions}"
-      moveit_active="${moveit_active}" />
+      low_level_mode="${low_level_mode}"
+      initial_positions="${initial_positions}" />
     <!-- Define material colors -->
     <material name="lightgray">

Commit message: Added modbus gripper communication in a separate thread to the low level hardware interface

File: link6_description/urdf/link6.ros2_control.xacro (robot description, xacro)
@@ -134,27 +134,4 @@
           <state_interface name="effort" />
         </joint>
-        <!-- If using the real robot, we need to define gripper joints for the hardware interface -->
-        <xacro:unless value="${use_fake_hardware or sim_gazebo}">
-          <xacro:unless value="${not gripper}">
-            <xacro:if value="${use_internal_bus_gripper_comm}">
-              <!-- Gripper A joint (only if gripper_joint_name is defined and not empty) -->
-              <xacro:unless value="${gripper_joint_name == '' or gripper_joint_name == None}">
-                <joint name="${prefix}${gripper_joint_name}">
-                  <command_interface name="position" />
-                  <state_interface name="position"/>
-                  <state_interface name="velocity"/>
-                </joint>
-              </xacro:unless>
-              <!-- Gripper B joint (only if gripper_b_joint_name is defined and not empty) -->
-              <xacro:unless value="${gripper_b_joint_name == '' or gripper_b_joint_name == None}">
-                <joint name="${prefix}${gripper_b_joint_name}">
-                  <command_interface name="position" />
-                  <state_interface name="position"/>
-                  <state_interface name="velocity"/>
-                </joint>
-              </xacro:unless>
-            </xacro:if>
-          </xacro:unless>
-        </xacro:unless>
       </xacro:unless>
       <xacro:if value="${low_level_mode}">
@@ -250,4 +227,27 @@
         </joint>
       </xacro:if>
+      <!-- If using the real robot, we need to define gripper joints for the hardware interface -->
+      <xacro:unless value="${use_fake_hardware or sim_gazebo}">
+        <xacro:unless value="${not gripper}">
+          <xacro:if value="${use_internal_bus_gripper_comm}">
+            <!-- Gripper A joint (only if gripper_joint_name is defined and not empty) -->
+            <xacro:unless value="${gripper_joint_name == '' or gripper_joint_name == None}">
+              <joint name="${prefix}${gripper_joint_name}">
+                <command_interface name="position" />
+                <state_interface name="position"/>
+                <state_interface name="velocity"/>
+              </joint>
+            </xacro:unless>
+            <!-- Gripper B joint (only if gripper_b_joint_name is defined and not empty) -->
+            <xacro:unless value="${gripper_b_joint_name == '' or gripper_b_joint_name == None}">
+              <joint name="${prefix}${gripper_b_joint_name}">
+                <command_interface name="position" />
+                <state_interface name="position"/>
+                <state_interface name="velocity"/>
+              </joint>
+            </xacro:unless>
+          </xacro:if>
+        </xacro:unless>
+      </xacro:unless>
     </ros2_control>
   </xacro:macro>
