Commit message: integrated dual gripper in robot macro

File: link6_description/urdf/link6_macro.xacro (robot description, xacro)
@@ -14,5 +14,6 @@
     sim_gazebo:=false
     initial_positions:=${dict(joint_1=0.0,joint_2=0.0,joint_3=0.0,joint_4=0.0,joint_5=0.0,joint_6=0.0)}
-    gripper_com_port:=/dev/ttyUSB0
+    gripper_com_port_left:=/dev/ttyUSB0
+    gripper_com_port_right:=/dev/ttyUSB1
     moveit_active:=false">
     <!-- ros2 control include -->
@@ -427,16 +428,15 @@
     <!-- Include and load the gripper if defined -->
     <xacro:unless value="${not gripper}">
-      <xacro:include filename="$(find robotiq_description)/urdf/robotiq_2f_85_macro.urdf.xacro" />
-      <xacro:robotiq_gripper
-        name="RobotiqGripperHardwareInterface"
+      <xacro:include filename="$(find agri_harveyl_description)/urdf/double_gripper_macro.urdf.xacro" />
+      <xacro:double_robotiq_gripper
         parent="${prefix}end_effector_link"
         prefix="${prefix}"
         use_fake_hardware="${use_fake_hardware}"
         fake_sensor_commands="${fake_sensor_commands}"
-        include_ros2_control="true"
-        com_port="${gripper_com_port}"
-        sim_ignition="${sim_gazebo}">
-        <origin xyz="0 0 0" rpy="0 0 0" />
-      </xacro:robotiq_gripper>
+        use_sim="${sim_gazebo}"
+        com_port_left="${gripper_com_port_left}"
+        com_port_right="${gripper_com_port_right}">
+        <origin xyz="0 0 0" rpy="0 0 0" />
+      </xacro:double_robotiq_gripper>
     </xacro:unless>
   </xacro:macro>

Commit message: Reverted back to single gripper.

File: link6_description/urdf/link6_macro.xacro (robot description, xacro)
@@ -428,4 +428,18 @@
     <!-- Include and load the gripper if defined -->
     <xacro:unless value="${not gripper}">
+      <xacro:include filename="$(find robotiq_description)/urdf/robotiq_2f_85_macro.urdf.xacro" />
+        <xacro:robotiq_gripper
+          name="RobotiqGripperHardwareInterface"
+          parent="${prefix}end_effector_link"
+          prefix="${prefix}"
+          use_fake_hardware="${use_fake_hardware}"
+          fake_sensor_commands="${fake_sensor_commands}"
+          include_ros2_control="false"
+          com_port="${gripper_com_port_left}"
+          sim_ignition="${sim_gazebo}">
+          <origin xyz="0 0 0" rpy="0 0 0" />
+        </xacro:robotiq_gripper>
+    </xacro:unless>
+    <!-- <xacro:unless value="${not gripper}">
       <xacro:include filename="$(find agri_harveyl_description)/urdf/double_gripper_macro.urdf.xacro" />
       <xacro:double_robotiq_gripper
@@ -439,5 +453,5 @@
         <origin xyz="0 0 0" rpy="0 0 0" />
       </xacro:double_robotiq_gripper>
-    </xacro:unless>
+    </xacro:unless> -->
   </xacro:macro>
 </robot>

Commit message: modular config seems to be working except single config is bugging. Instant stalling. Dont know why yet.

File: link6_description/urdf/link6_macro.xacro (robot description, xacro)
@@ -17,4 +17,7 @@
     gripper_com_port_right:=/dev/ttyUSB1
     moveit_active:=false">
+    <!-- Available grippers defined here -->
+    <xacro:property name="available_grippers" value="['robotiq_2f_85', 'double_gripper']"/>
+    <xacro:property name="PI" value="3.14159"/>
     <!-- ros2 control include -->
     <xacro:include filename="$(find link6_description)/urdf/link6.ros2_control.xacro" />
@@ -416,30 +419,19 @@
       <child link="${prefix}end_effector_link" />
     </joint>
-    <!-- If no gripper, define tool frame here -->
-    <xacro:if value="${not gripper}">
-      <link name="${prefix}tool_frame" />
-      <joint name="${prefix}tool_frame_joint" type="fixed">
-        <origin xyz="0 0 0" rpy="0 0 0" />
-        <parent link="${prefix}end_effector_link" />
-        <child link="${prefix}tool_frame" />
-        <axis xyz="0 0 0" />
-      </joint>
-    </xacro:if>
-    <!-- Include and load the gripper if defined -->
-    <xacro:unless value="${not gripper}">
+    <!-- Include and load gripper logic based off of available grippers for link_6 -->
+    <xacro:if value="${gripper == 'robotiq_2f_85'}">
       <xacro:include filename="$(find robotiq_description)/urdf/robotiq_2f_85_macro.urdf.xacro" />
         <xacro:robotiq_gripper
-          name="RobotiqGripperHardwareInterface"
+          name="robotiq_single_gripper"
           parent="${prefix}end_effector_link"
           prefix="${prefix}"
           use_fake_hardware="${use_fake_hardware}"
           fake_sensor_commands="${fake_sensor_commands}"
-          include_ros2_control="false"
           com_port="${gripper_com_port_left}"
           sim_ignition="${sim_gazebo}">
-          <origin xyz="0 0 0" rpy="0 0 0" />
+          <origin xyz="0 0 0.05" rpy="${PI/4} 0 0" />
         </xacro:robotiq_gripper>
-    </xacro:unless>
-    <!-- <xacro:unless value="${not gripper}">
+    </xacro:if>
+    <xacro:if value="${gripper == 'double_gripper'}">
       <xacro:include filename="$(find agri_harveyl_description)/urdf/double_gripper_macro.urdf.xacro" />
       <xacro:double_robotiq_gripper
@@ -453,5 +445,15 @@
         <origin xyz="0 0 0" rpy="0 0 0" />
       </xacro:double_robotiq_gripper>
-    </xacro:unless> -->
+    </xacro:if>
+    <!-- If no gripper, define tool frame here -->
+    <xacro:if value="${gripper == ''}">
+      <link name="${prefix}tool_frame" />
+      <joint name="${prefix}tool_frame_joint" type="fixed">
+        <origin xyz="0 0 0" rpy="0 0 0" />
+        <parent link="${prefix}end_effector_link" />
+        <child link="${prefix}tool_frame" />
+        <axis xyz="0 0 0" />
+      </joint>
+    </xacro:if>
   </xacro:macro>
 </robot>

Commit message: Reduced Link6 collision radius

File: link6_description/urdf/link6_macro.xacro (robot description, xacro)
@@ -17,4 +17,12 @@
     gripper_com_port_right:=/dev/ttyUSB1
     moveit_active:=false">
+    <!-- Properties -->
+    <xacro:property name="base_collision_radius" value="0.08"/>
+    <xacro:property name="shoulder_collision_radius" value="0.07"/>
+    <xacro:property name="arm_collision_radius" value="0.06"/>
+    <xacro:property name="forearm_collision_radius" value="0.055"/>
+    <xacro:property name="lower_wrist_collision_radius" value="0.05"/>
+    <xacro:property name="upper_wrist_collision_radius" value="0.05"/>
+    <xacro:property name="wrist_interface_collision_radius" value="0.05"/>
     <!-- ros2 control include -->
     <xacro:include filename="$(find link6_description)/urdf/link6.ros2_control.xacro" />
@@ -62,5 +70,5 @@
         <origin xyz="0 0 0" rpy="0 0 0" />
         <geometry>
-          <sphere radius="0.1" />
+          <sphere radius="${base_collision_radius}" />
         </geometry>
       </collision>
@@ -83,5 +91,5 @@
         <origin xyz="0 0 -0.04" rpy="0 0 0" />
         <geometry>
-          <sphere radius="0.09" />
+          <sphere radius="${shoulder_collision_radius}" />
         </geometry>
       </collision>
@@ -89,5 +97,5 @@
         <origin xyz="0.06065737 -0.01 -0.08144986" rpy="0 0 0" />
         <geometry>
-          <sphere radius="0.095" />
+          <sphere radius="${shoulder_collision_radius}" />
         </geometry>
       </collision>
@@ -95,5 +103,5 @@
         <origin xyz="0 0 -0.11" rpy="0 0 0" />
         <geometry>
-          <sphere radius="0.09" />
+          <sphere radius="${shoulder_collision_radius}" />
         </geometry>
       </collision>
@@ -101,5 +109,5 @@
         <origin xyz="0.1078564 -0.02138667 -0.1392602" rpy="0 0 0" />
         <geometry>
-          <sphere radius="0.095" />
+          <sphere radius="${shoulder_collision_radius}" />
         </geometry>
       </collision>
@@ -107,5 +115,5 @@
         <origin xyz="0.04343076 -0.003456797 -0.1306261" rpy="0 0 0" />
         <geometry>
-          <sphere radius="0.095" />
+          <sphere radius="${shoulder_collision_radius}" />
         </geometry>
       </collision>
@@ -136,5 +144,5 @@
         <origin xyz="0 0 -0.01524985" rpy="0 0 0" />
         <geometry>
-          <sphere radius="0.08" />
+          <sphere radius="${arm_collision_radius}" />
         </geometry>
       </collision>
@@ -142,5 +150,5 @@
         <origin xyz="0 0.003107564 -0.05411892" rpy="0 0 0" />
         <geometry>
-          <sphere radius="0.085" />
+          <sphere radius="${arm_collision_radius}" />
         </geometry>
       </collision>
@@ -148,5 +156,5 @@
         <origin xyz="0 0.04674223 -0.07957917" rpy="0 0 0" />
         <geometry>
-          <sphere radius="0.08" />
+          <sphere radius="${arm_collision_radius}" />
         </geometry>
       </collision>
@@ -154,5 +162,5 @@
         <origin xyz="0 0.1114492 -0.07957917" rpy="0 0 0" />
         <geometry>
-          <sphere radius="0.08" />
+          <sphere radius="${arm_collision_radius}" />
         </geometry>
       </collision>
@@ -160,5 +168,5 @@
         <origin xyz="0 0.179992  -0.07957917" rpy="0 0 0" />
         <geometry>
-          <sphere radius="0.08" />
+          <sphere radius="${arm_collision_radius}" />
         </geometry>
       </collision>
@@ -166,5 +174,5 @@
         <origin xyz="0 0.2487042 -0.07957917" rpy="0 0 0" />
         <geometry>
-          <sphere radius="0.08" />
+          <sphere radius="${arm_collision_radius}" />
         </geometry>
       </collision>
@@ -172,5 +180,5 @@
         <origin xyz="0 0.3173259 -0.07957917" rpy="0 0 0" />
         <geometry>
-          <sphere radius="0.08" />
+          <sphere radius="${arm_collision_radius}" />
         </geometry>
       </collision>
@@ -178,5 +186,5 @@
         <origin xyz="0 0.3835145 -0.07957917" rpy="0 0 0" />
         <geometry>
-          <sphere radius="0.08" />
+          <sphere radius="${arm_collision_radius}" />
         </geometry>
       </collision>
@@ -184,5 +192,5 @@
         <origin xyz="0 0.4415521 -0.07957917" rpy="0 0 0" />
         <geometry>
-          <sphere radius="0.08" />
+          <sphere radius="${arm_collision_radius}" />
         </geometry>
       </collision>
@@ -190,5 +198,5 @@
         <origin xyz="0 0.4824647 -0.05411892" rpy="0 0 0" />
         <geometry>
-          <sphere radius="0.085" />
+          <sphere radius="${arm_collision_radius}" />
         </geometry>
       </collision>
@@ -196,5 +204,5 @@
         <origin xyz="0 0.4848319 -0.01524985" rpy="0 0 0" />
         <geometry>
-          <sphere radius="0.08" />
+          <sphere radius="${arm_collision_radius}" />
         </geometry>
       </collision>
@@ -225,5 +233,5 @@
         <origin xyz="0 0 -0.01478543" rpy="0 0 0" />
         <geometry>
-          <sphere radius="0.08" />
+          <sphere radius="${forearm_collision_radius}" />
         </geometry>
       </collision>
@@ -231,5 +239,5 @@
         <origin xyz="0 -0.002774531 -0.05402248" rpy="0 0 0" />
         <geometry>
-          <sphere radius="0.085" />
+          <sphere radius="${forearm_collision_radius}" />
         </geometry>
       </collision>
@@ -237,5 +245,5 @@
         <origin xyz="0 -0.02792384  -0.08310601" rpy="0 0 0" />
         <geometry>
-          <sphere radius="0.08" />
+          <sphere radius="${forearm_collision_radius}" />
         </geometry>
       </collision>
@@ -243,5 +251,5 @@
         <origin xyz="0 -0.07494865 -0.09085903" rpy="0 0 0" />
         <geometry>
-          <sphere radius="0.075" />
+          <sphere radius="${forearm_collision_radius}" />
         </geometry>
       </collision>
@@ -249,5 +257,5 @@
         <origin xyz="0 -0.1212274  -0.091767" rpy="0 0 0" />
         <geometry>
-          <sphere radius="0.075" />
+          <sphere radius="${forearm_collision_radius}" />
         </geometry>
       </collision>
@@ -279,5 +287,5 @@
         <origin xyz="0 0 -0.01025881" rpy="0 0 0" />
         <geometry>
-          <sphere radius="0.07" />
+          <sphere radius="${lower_wrist_collision_radius}" />
         </geometry>
       </collision>
@@ -285,5 +293,5 @@
         <origin xyz="0 0 -0.06014508" rpy="0 0 0" />
         <geometry>
-          <sphere radius="0.07" />
+          <sphere radius="${lower_wrist_collision_radius}" />
         </geometry>
       </collision>
@@ -291,5 +299,5 @@
         <origin xyz="0 0 -0.1106502" rpy="0 0 0" />
         <geometry>
-          <sphere radius="0.07" />
+          <sphere radius="${lower_wrist_collision_radius}" />
         </geometry>
       </collision>
@@ -297,5 +305,5 @@
         <origin xyz="0 0 -0.1607216" rpy="0 0 0" />
         <geometry>
-          <sphere radius="0.07" />
+          <sphere radius="${lower_wrist_collision_radius}" />
         </geometry>
       </collision>
@@ -303,5 +311,5 @@
         <origin xyz="0 -0.001607588 -0.2100781" rpy="0 0 0" />
         <geometry>
-          <sphere radius="0.07" />
+          <sphere radius="${lower_wrist_collision_radius}" />
         </geometry>
       </collision>
@@ -309,5 +317,5 @@
         <origin xyz="0 -0.03559661 -0.222183" rpy="0 0 0" />
         <geometry>
-          <sphere radius="0.07" />
+          <sphere radius="${lower_wrist_collision_radius}" />
         </geometry>
       </collision>
@@ -339,5 +347,5 @@
         <origin xyz="0 0 -0.02579783" rpy="0 0 0" />
         <geometry>
-          <sphere radius="0.07" />
+          <sphere radius="${upper_wrist_collision_radius}" />
         </geometry>
       </collision>
@@ -345,5 +353,5 @@
         <origin xyz="0 0 -0.06192018" rpy="0 0 0" />
         <geometry>
-          <sphere radius="0.07" />
+          <sphere radius="${upper_wrist_collision_radius}" />
         </geometry>
       </collision>
@@ -351,5 +359,5 @@
         <origin xyz="0.00760242 0.03851649 -0.07210818" rpy="0 0 0" />
         <geometry>
-          <sphere radius="0.075" />
+          <sphere radius="${upper_wrist_collision_radius}" />
         </geometry>
       </collision>
@@ -357,5 +365,5 @@
         <origin xyz="0.01731829 0.07948508 -0.07309098" rpy="0 0 0" />
         <geometry>
-          <sphere radius="0.075" />
+          <sphere radius="${upper_wrist_collision_radius}" />
         </geometry>
       </collision>
@@ -363,5 +371,5 @@
         <origin xyz="0.06120646 0.0860149 -0.07708402" rpy="0 0 0" />
         <geometry>
-          <sphere radius="0.07" />
+          <sphere radius="${upper_wrist_collision_radius}" />
         </geometry>
       </collision>
@@ -392,5 +400,5 @@
         <origin xyz="0 0 -0.02647703" rpy="0 0 0" />
         <geometry>
-          <sphere radius="0.07" />
+          <sphere radius="${wrist_interface_collision_radius}" />
         </geometry>
       </collision>
@@ -398,5 +406,5 @@
         <origin xyz="0 0 -0.06063214" rpy="0 0 0" />
         <geometry>
-          <sphere radius="0.07" />
+          <sphere radius="${wrist_interface_collision_radius}" />
         </geometry>
       </collision>

Commit message: Added a tool_frame for the robotiq_2f_85 gripper

File: link6_description/urdf/link6_macro.xacro (robot description, xacro)
@@ -437,6 +437,12 @@
         com_port="${gripper_com_port_left}"
         sim_ignition="${sim_gazebo}">
-        <origin xyz="0 0 0" rpy="0 0 0" />
+        <origin xyz="0 0 0" rpy="0 0 3.14159" />
       </xacro:robotiq_gripper>
+      <link name="${prefix}tool_frame"></link>
+      <joint name="${prefix}tool_frame_joint" type="fixed">
+          <origin xyz="0 0 0.12" rpy="0 0 0"/>
+          <parent link="${prefix}robotiq_85_base_link"/>
+          <child link="${prefix}tool_frame"/>
+      </joint>
     </xacro:if>
     <xacro:if value="${gripper == 'double_robotiq'}">

Commit message: Fixed issue in arm macro when simulating with a gripper, added moveit usage instructions

File: link6_description/urdf/link6_macro.xacro (robot description, xacro)
@@ -14,6 +14,5 @@
     sim_gazebo:=false
     initial_positions:=${dict(joint_1=0.0,joint_2=0.0,joint_3=0.0,joint_4=0.0,joint_5=0.0,joint_6=0.0)}
-    gripper_com_port_left:=/dev/ttyUSB0
-    gripper_com_port_right:=/dev/ttyUSB1
+    gripper_com_port:=/dev/ttyUSB0
     moveit_active:=false">
     <!-- Properties -->
@@ -443,23 +442,10 @@
           use_fake_hardware="${use_fake_hardware}"
           fake_sensor_commands="${fake_sensor_commands}"
-          include_ros2_control="false"
-          com_port="${gripper_com_port_left}"
+          include_ros2_control="${sim_gazebo}"
+          com_port="${gripper_com_port}"
           sim_ignition="${sim_gazebo}">
           <origin xyz="0 0 0" rpy="0 0 0" />
         </xacro:robotiq_gripper>
     </xacro:unless>
-    <!-- <xacro:unless value="${not gripper}">
-      <xacro:include filename="$(find agri_harveyl_description)/urdf/double_gripper_macro.urdf.xacro" />
-      <xacro:double_robotiq_gripper
-        parent="${prefix}end_effector_link"
-        prefix="${prefix}"
-        use_fake_hardware="${use_fake_hardware}"
-        fake_sensor_commands="${fake_sensor_commands}"
-        use_sim="${sim_gazebo}"
-        com_port_left="${gripper_com_port_left}"
-        com_port_right="${gripper_com_port_right}">
-        <origin xyz="0 0 0" rpy="0 0 0" />
-      </xacro:double_robotiq_gripper>
-    </xacro:unless> -->
   </xacro:macro>
 </robot>

Commit message: Removed gripper macros from the link6 macro, removed gripper urdf files

File: link6_description/urdf/link6_macro.xacro (robot description, xacro)
@@ -416,82 +416,4 @@
       <child link="${prefix}end_effector_link" />
     </joint>
-    <!-- If no gripper, define tool frame here -->
-    <xacro:if value="${gripper == ''}">
-      <link name="${prefix}tool_frame" />
-      <joint name="${prefix}tool_frame_joint" type="fixed">
-        <origin xyz="0 0 0" rpy="0 0 0" />
-        <parent link="${prefix}end_effector_link" />
-        <child link="${prefix}tool_frame" />
-        <axis xyz="0 0 0" />
-      </joint>
-    </xacro:if>
-    <!-- Include and load gripper based on available grippers for Link6 -->
-    <xacro:if value="${gripper == 'robotiq_2f_85'}">
-      <xacro:include filename="$(find robotiq_description)/urdf/robotiq_2f_85_macro.urdf.xacro" />
-      <xacro:robotiq_gripper
-        name="RobotiqGripperHardwareInterface"
-        parent="${prefix}end_effector_link"
-        prefix="${prefix}"
-        use_fake_hardware="${use_fake_hardware}"
-        fake_sensor_commands="${fake_sensor_commands}"
-        include_ros2_control="${sim_gazebo}"
-        com_port="${gripper_com_port_left}"
-        sim_ignition="${sim_gazebo}">
-        <origin xyz="0 0 0" rpy="0 0 3.14159" />
-      </xacro:robotiq_gripper>
-      <link name="${prefix}tool_frame"></link>
-      <joint name="${prefix}tool_frame_joint" type="fixed">
-          <origin xyz="0 0 0.12" rpy="0 0 0"/>
-          <parent link="${prefix}robotiq_85_base_link"/>
-          <child link="${prefix}tool_frame"/>
-      </joint>
-    </xacro:if>
-    <xacro:if value="${gripper == 'robotiq_hande'}">
-      <xacro:include filename="$(find link6_description)/urdf/robotiq_hande_cutter.xacro" />
-      <xacro:robotiq_hande_gripper
-          name="RobotiqGripperHardwareInterface"
-          prefix="${prefix}"
-          parent="${prefix}end_effector_link"
-          grip_pos_min="0"
-          grip_pos_max="0.025"
-          tty_port="${gripper_com_port_left}"
-          baudrate="115200"
-          parity="N"
-          data_bits="8"
-          stop_bit="1"
-          slave_id="9"
-          use_fake_hardware="${use_fake_hardware}"
-          include_ros2_control="${sim_gazebo}"
-          sim_gazebo="${sim_gazebo}"
-          xyz="0 0 0"
-          rpy="0 0 3.14159"
-      />
-    </xacro:if>
-    <xacro:if value="${gripper == 'double_robotiq'}">
-      <xacro:include filename="$(find link6_description)/urdf/double_robotiq_macro.urdf.xacro" />
-      <xacro:double_robotiq_gripper
-        parent="${prefix}end_effector_link"
-        prefix="${prefix}"
-        use_fake_hardware="${use_fake_hardware}"
-        fake_sensor_commands="${fake_sensor_commands}"
-        use_sim="${sim_gazebo}"
-        com_port_left="${gripper_com_port_left}"
-        com_port_right="${gripper_com_port_right}">
-        <origin xyz="0 0 0" rpy="0 0 0" />
-      </xacro:double_robotiq_gripper>
-    </xacro:if>
-    <xacro:if value="${gripper == 'double_robotiq_90'}">
-      <xacro:include filename="$(find link6_description)/urdf/double_robotiq_90_macro.urdf.xacro" />
-      <xacro:double_robotiq_gripper_90
-        parent="${prefix}end_effector_link"
-        prefix="${prefix}"
-        use_fake_hardware="${use_fake_hardware}"
-        fake_sensor_commands="${fake_sensor_commands}"
-        use_sim="${sim_gazebo}"
-        com_port_left="${gripper_com_port_left}"
-        com_port_right="${gripper_com_port_right}">
-        <origin xyz="0 0 0" rpy="0 0 0" />
-      </xacro:double_robotiq_gripper_90>
-    </xacro:if>
   </xacro:macro>
 </robot>
